Commit message: Add materilas.xacro file

File: src/volcaniarm_description/urdf/materials.xacro (robot description, xacro)
@@ -17,5 +17,5 @@
   </material>
   <material name="grey">
-    <color rgba="0.5 0.5 0.5 1.0"/>
+    <color rgba="0.75 0.75 0.8 1.0"/>
   </material>
   <material name="orange">

File: src/volcaniarm_description/urdf/volcaniarm.xacro (robot description, xacro)
@@ -1,4 +1,6 @@
 <?xml version="1.0"?>
 <robot xmlns:xacro="http://www.ros.org/wiki/xacro" name="volcaniarm">
+  <!-- Include materials -->
+  <xacro:include filename="$(find volcaniarm_description)/urdf/materials.xacro"/>
   <!-- World link (fixed reference frame) -->
   <link name="world"/>
@@ -22,7 +24,5 @@
         <mesh filename="package://volcaniarm_description/meshes/volcaniarm_base_link.STL"/>
       </geometry>
-      <material name="">
-        <color rgba="0.792156862745098 0.819607843137255 0.933333333333333 1"/>
-      </material>
+      <material name="grey"/>
     </visual>
     <collision>
@@ -46,7 +46,5 @@
         <mesh filename="package://volcaniarm_description/meshes/delta_arm_base_link.STL"/>
       </geometry>
-      <material name="">
-        <color rgba="0.792156862745098 0.819607843137255 0.933333333333333 1"/>
-      </material>
+      <material name="grey"/>
     </visual>
     <collision>
@@ -77,7 +75,5 @@
         <mesh filename="package://volcaniarm_description/meshes/right_elbow_link.STL"/>
       </geometry>
-      <material name="">
-        <color rgba="0.792156862745098 0.819607843137255 0.933333333333333 1"/>
-      </material>
+      <material name="grey"/>
     </visual>
     <collision>
@@ -108,7 +104,5 @@
         <mesh filename="package://volcaniarm_description/meshes/left_elbow_link.STL"/>
       </geometry>
-      <material name="">
-        <color rgba="0.792156862745098 0.819607843137255 0.933333333333333 1"/>
-      </material>
+      <material name="grey"/>
     </visual>
     <collision>
@@ -126,5 +120,5 @@
     <limit lower="-1.57" upper="1.57" effort="0" velocity="0"/>
   </joint>
-  <!-- right_arm_link
+  <!-- right_arm_link -->
   <link name="right_arm_link">
     <inertial>
@@ -139,7 +133,5 @@
         <mesh filename="package://volcaniarm_description/meshes/right_arm_link.STL"/>
       </geometry>
-      <material name="">
-        <color rgba="0.792156862745098 0.819607843137255 0.933333333333333 1"/>
-      </material>
+      <material name="grey"/>
     </visual>
     <collision>
@@ -156,7 +148,7 @@
     <axis xyz="-1 0 0"/>
     <limit lower="-1.57" upper="1.57" effort="10" velocity="10"/>
-  </joint> -->
+  </joint>
   <!-- left_arm_link -->
-  <!-- <link name="left_arm_link">
+  <link name="left_arm_link">
     <inertial>
       <origin xyz="0.0017145275657231 2.87547763377916E-13 0.231024142798437" rpy="0 0 0"/>
@@ -170,7 +162,5 @@
         <mesh filename="package://volcaniarm_description/meshes/left_arm_link.STL"/>
       </geometry>
-      <material name="">
-        <color rgba="0.792156862745098 0.819607843137255 0.933333333333333 1"/>
-      </material>
+      <material name="grey"/>
     </visual>
     <collision>
@@ -187,4 +177,4 @@
     <axis xyz="1 0 0"/>
     <limit lower="-1.57" upper="1.57" effort="0" velocity="0"/>
-  </joint> -->
+  </joint>
 </robot>
