Commit message: description: real-robot palette via named materials (matches Isaac PBR base colors)

File: src/volcaniarm_description/urdf/materials.xacro (robot description, xacro)
@@ -1,27 +1,37 @@
 <?xml version="1.0"?>
-<robot>
-  <material name="black">
-    <color rgba="0.0 0.0 0.0 1.0"/>
+<!-- Real-robot flat-color palette — the single source of visual colors for
+     RViz and Gazebo. Each color exists twice on purpose:
+       * a xacro property (so visuals can inline the rgba — libsdformat and
+         the Isaac URDF importer don't reliably resolve named-material
+         references, RViz does)
+       * a named <material> (so RViz shows a meaningful name)
+     Keep the RGB values in sync with the PBR palette in
+     volcaniarm_isaaclab/scripts/apply_materials.py (MATERIAL_GROUPS
+     base_color) — that script is what colors the Isaac Sim USD; these flat
+     values are its RViz/Gazebo approximation. -->
+<robot xmlns:xacro="http://www.ros.org/wiki/xacro">
+  <!-- Powder-coated red table frame (base_link + table legs). -->
+  <xacro:property name="powder_red_rgba" value="0.62 0.07 0.09 1.0"/>
+  <material name="powder_red">
+    <color rgba="${powder_red_rgba}"/>
   </material>
-  <material name="white">
-    <color rgba="1.0 1.0 1.0 1.0"/>
+  <!-- Cool galvanized steel (arm links, camera, casters). -->
+  <xacro:property name="galvanized_rgba" value="0.72 0.74 0.76 1.0"/>
+  <material name="galvanized">
+    <color rgba="${galvanized_rgba}"/>
   </material>
-  <material name="red">
-    <color rgba="0.8 0.0 0.0 1.0"/>
+  <!-- Painted black steel (arm mounting column). -->
+  <xacro:property name="steel_black_rgba" value="0.02 0.02 0.02 1.0"/>
+  <material name="steel_black">
+    <color rgba="${steel_black_rgba}"/>
   </material>
-  <material name="blue">
-    <color rgba="0.0 0.0 0.8 1.0"/>
+  <!-- Matte black printed plastic (camera rev mount). -->
+  <xacro:property name="plastic_black_rgba" value="0.04 0.04 0.04 1.0"/>
+  <material name="plastic_black">
+    <color rgba="${plastic_black_rgba}"/>
   </material>
-  <material name="green">
-    <color rgba="0.0 0.8 0.0 1.0"/>
-  </material>
-  <material name="grey">
-    <color rgba="0.75 0.75 0.8 1.0"/>
-  </material>
-  <material name="orange">
-    <color rgba="${255/255} ${108/255} ${10/255} 1.0"/>
-  </material>
-  <material name="brown">
-    <color rgba="${222/255} ${207/255} ${195/255} 1.0"/>
-  </material>
+  <!-- Debug-visual colors (closure scaffolding spheres — sim-side aids,
+       stripped from the Isaac URDF by sync_urdf.py). -->
+  <xacro:property name="tip_green_rgba" value="0.0 1.0 0.0 1.0"/>
+  <xacro:property name="closure_purple_rgba" value="0.6 0.0 0.8 1.0"/>
 </robot>

File: src/volcaniarm_description/urdf/volcaniarm.urdf.xacro (robot description, xacro)
@@ -47,4 +47,6 @@
   <xacro:property name="camera_mount_x" value="$(arg camera_mount_x)" />
   <xacro:property name="camera_mount_pitch" value="$(arg camera_mount_pitch)" />
+  <!-- Real-robot color palette (named materials + rgba properties). -->
+  <xacro:include filename="$(find volcaniarm_description)/urdf/materials.xacro" />
    <!-- ros2_control hardware interfaces -->
   <xacro:include filename="$(find volcaniarm_description)/urdf/volcaniarm_ros2_control.xacro" />
@@ -97,6 +99,6 @@
         <mesh filename="package://volcaniarm_description/meshes/base_link.STL" />
       </geometry>
-      <material name="">
-        <color rgba="1 0 0 1" />
+      <material name="powder_red">
+        <color rgba="${powder_red_rgba}" />
       </material>
     </visual>
@@ -122,6 +124,6 @@
         <mesh filename="package://volcaniarm_description/meshes/fl_table_leg_link.STL" />
       </geometry>
-      <material name="">
-        <color rgba="0.79216 0.81961 0.93333 1" />
+      <material name="powder_red">
+        <color rgba="${powder_red_rgba}" />
       </material>
     </visual>
@@ -151,6 +153,6 @@
         <mesh filename="package://volcaniarm_description/meshes/fl_caster_wheel_mount_link.STL" />
       </geometry>
-      <material name="">
-        <color rgba="0.79216 0.81961 0.93333 1" />
+      <material name="galvanized">
+        <color rgba="${galvanized_rgba}" />
       </material>
     </visual>
@@ -180,6 +182,6 @@
         <mesh filename="package://volcaniarm_description/meshes/fl_caster_wheel_link.STL" />
       </geometry>
-      <material name="">
-        <color rgba="0.79216 0.81961 0.93333 1" />
+      <material name="galvanized">
+        <color rgba="${galvanized_rgba}" />
       </material>
     </visual>
@@ -209,6 +211,6 @@
         <mesh filename="package://volcaniarm_description/meshes/fr_table_leg_link.STL" />
       </geometry>
-      <material name="">
-        <color rgba="0.79216 0.81961 0.93333 1" />
+      <material name="powder_red">
+        <color rgba="${powder_red_rgba}" />
       </material>
     </visual>
@@ -238,6 +240,6 @@
         <mesh filename="package://volcaniarm_description/meshes/fr_caster_wheel_mount_link.STL" />
       </geometry>
-      <material name="">
-        <color rgba="0.79216 0.81961 0.93333 1" />
+      <material name="galvanized">
+        <color rgba="${galvanized_rgba}" />
       </material>
     </visual>
@@ -267,6 +269,6 @@
         <mesh filename="package://volcaniarm_description/meshes/fr_caster_wheel_link.STL" />
       </geometry>
-      <material name="">
-        <color rgba="0.79216 0.81961 0.93333 1" />
+      <material name="galvanized">
+        <color rgba="${galvanized_rgba}" />
       </material>
     </visual>
@@ -296,6 +298,6 @@
         <mesh filename="package://volcaniarm_description/meshes/rl_table_leg_link.STL" />
       </geometry>
-      <material name="">
-        <color rgba="0.79216 0.81961 0.93333 1" />
+      <material name="powder_red">
+        <color rgba="${powder_red_rgba}" />
       </material>
     </visual>
@@ -325,6 +327,6 @@
         <mesh filename="package://volcaniarm_description/meshes/rl_caster_wheel_mount_link.STL" />
       </geometry>
-      <material name="">
-        <color rgba="0.79216 0.81961 0.93333 1" />
+      <material name="galvanized">
+        <color rgba="${galvanized_rgba}" />
       </material>
     </visual>
@@ -354,6 +356,6 @@
         <mesh filename="package://volcaniarm_description/meshes/rl_caster_wheel_link.STL" />
       </geometry>
-      <material name="">
-        <color rgba="0.79216 0.81961 0.93333 1" />
+      <material name="galvanized">
+        <color rgba="${galvanized_rgba}" />
       </material>
     </visual>
@@ -383,6 +385,6 @@
         <mesh filename="package://volcaniarm_description/meshes/rr_table_leg_link.STL" />
       </geometry>
-      <material name="">
-        <color rgba="0.79216 0.81961 0.93333 1" />
+      <material name="powder_red">
+        <color rgba="${powder_red_rgba}" />
       </material>
     </visual>
@@ -412,6 +414,6 @@
         <mesh filename="package://volcaniarm_description/meshes/rr_caster_wheel_mount_link.STL" />
       </geometry>
-      <material name="">
-        <color rgba="0.79216 0.81961 0.93333 1" />
+      <material name="galvanized">
+        <color rgba="${galvanized_rgba}" />
       </material>
     </visual>
@@ -441,6 +443,6 @@
         <mesh filename="package://volcaniarm_description/meshes/rr_caster_wheel_link.STL" />
       </geometry>
-      <material name="">
-        <color rgba="0.79216 0.81961 0.93333 1" />
+      <material name="galvanized">
+        <color rgba="${galvanized_rgba}" />
       </material>
     </visual>
@@ -470,6 +472,6 @@
         <mesh filename="package://volcaniarm_description/meshes/volcaniarm_base_link.STL" />
       </geometry>
-      <material name="">
-        <color rgba="0.79216 0.81961 0.93333 1" />
+      <material name="steel_black">
+        <color rgba="${steel_black_rgba}" />
       </material>
     </visual>
@@ -499,6 +501,6 @@
         <mesh filename="package://volcaniarm_description/meshes/volcaniarm_left_elbow_link.STL" />
       </geometry>
-      <material name="">
-        <color rgba="0.79216 0.81961 0.93333 1" />
+      <material name="galvanized">
+        <color rgba="${galvanized_rgba}" />
       </material>
     </visual>
@@ -530,6 +532,6 @@
         <mesh filename="package://volcaniarm_description/meshes/volcaniarm_left_arm_link.STL" />
       </geometry>
-      <material name="">
-        <color rgba="0.79216 0.81961 0.93333 1" />
+      <material name="galvanized">
+        <color rgba="${galvanized_rgba}" />
       </material>
     </visual>
@@ -562,6 +564,6 @@
         <mesh filename="package://volcaniarm_description/meshes/volcaniarm_right_elbow_link.STL" />
       </geometry>
-      <material name="">
-        <color rgba="0.79216 0.81961 0.93333 1" />
+      <material name="galvanized">
+        <color rgba="${galvanized_rgba}" />
       </material>
     </visual>
@@ -593,6 +595,6 @@
         <mesh filename="package://volcaniarm_description/meshes/volcaniarm_right_arm_link.STL" />
       </geometry>
-      <material name="">
-        <color rgba="0.79216 0.81961 0.93333 1" />
+      <material name="galvanized">
+        <color rgba="${galvanized_rgba}" />
       </material>
     </visual>
@@ -631,6 +633,6 @@
         <mesh filename="package://volcaniarm_description/meshes/camera_mount_linear_link.STL" />
       </geometry>
-      <material name="">
-        <color rgba="1 1 1 1" />
+      <material name="galvanized">
+        <color rgba="${galvanized_rgba}" />
       </material>
     </visual>
@@ -659,6 +661,6 @@
         <mesh filename="package://volcaniarm_description/meshes/camera_mount_rev_link.STL" />
       </geometry>
-      <material name="">
-        <color rgba="0.79216 0.81961 0.93333 1" />
+      <material name="plastic_black">
+        <color rgba="${plastic_black_rgba}" />
       </material>
     </visual>
@@ -690,6 +692,6 @@
         <mesh filename="package://volcaniarm_description/meshes/camera_link.STL" />
       </geometry>
-      <material name="">
-        <color rgba="0.79216 0.81961 0.93333 1" />
+      <material name="galvanized">
+        <color rgba="${galvanized_rgba}" />
       </material>
     </visual>
@@ -737,5 +739,5 @@
       </geometry>
       <material name="tip_green">
-        <color rgba="0.0 1.0 0.0 1.0" />
+        <color rgba="${tip_green_rgba}" />
       </material>
     </visual>
@@ -769,5 +771,5 @@
       </geometry>
       <material name="closure_purple">
-        <color rgba="0.6 0.0 0.8 1.0" />
+        <color rgba="${closure_purple_rgba}" />
       </material>
     </visual>

Commit message: materials: anonymous inline colors (named root materials made RViz paint the whole robot one color)

File: src/volcaniarm_description/urdf/materials.xacro (robot description, xacro)
@@ -1,9 +1,10 @@
 <?xml version="1.0"?>
 <!-- Real-robot flat-color palette — the single source of visual colors for
-     RViz and Gazebo. Each color exists twice on purpose:
-       * a xacro property (so visuals can inline the rgba — libsdformat and
-         the Isaac URDF importer don't reliably resolve named-material
-         references, RViz does)
-       * a named <material> (so RViz shows a meaningful name)
+     RViz and Gazebo, as xacro rgba properties that visuals inline into
+     ANONYMOUS <material name=""> tags. Deliberately no named/root-level
+     <material> definitions: RViz's urdf material resolver maps materials
+     by name and repaints every referencing link with one entry (whole
+     robot rendered a single color), while anonymous inline colors render
+     correctly in RViz, libsdformat/gz, and the Isaac URDF importer alike.
      Keep the RGB values in sync with the PBR palette in
      volcaniarm_isaaclab/scripts/apply_materials.py (MATERIAL_GROUPS
@@ -13,22 +14,10 @@
   <!-- Powder-coated red table frame (base_link + table legs). -->
   <xacro:property name="powder_red_rgba" value="0.62 0.07 0.09 1.0"/>
-  <material name="powder_red">
-    <color rgba="${powder_red_rgba}"/>
-  </material>
   <!-- Cool galvanized steel (arm links, camera, casters). -->
   <xacro:property name="galvanized_rgba" value="0.72 0.74 0.76 1.0"/>
-  <material name="galvanized">
-    <color rgba="${galvanized_rgba}"/>
-  </material>
   <!-- Painted black steel (arm mounting column). -->
   <xacro:property name="steel_black_rgba" value="0.02 0.02 0.02 1.0"/>
-  <material name="steel_black">
-    <color rgba="${steel_black_rgba}"/>
-  </material>
   <!-- Matte black printed plastic (camera rev mount). -->
   <xacro:property name="plastic_black_rgba" value="0.04 0.04 0.04 1.0"/>
-  <material name="plastic_black">
-    <color rgba="${plastic_black_rgba}"/>
-  </material>
   <!-- Debug-visual colors (closure scaffolding spheres — sim-side aids,
        stripped from the Isaac URDF by sync_urdf.py). -->

File: src/volcaniarm_description/urdf/volcaniarm.urdf.xacro (robot description, xacro)
@@ -47,5 +47,6 @@
   <xacro:property name="camera_mount_x" value="$(arg camera_mount_x)" />
   <xacro:property name="camera_mount_pitch" value="$(arg camera_mount_pitch)" />
-  <!-- Real-robot color palette (named materials + rgba properties). -->
+  <!-- Real-robot color palette (rgba xacro properties, inlined anonymously
+       into each visual — see materials.xacro for why not named). -->
   <xacro:include filename="$(find volcaniarm_description)/urdf/materials.xacro" />
    <!-- ros2_control hardware interfaces -->
@@ -99,5 +100,5 @@
         <mesh filename="package://volcaniarm_description/meshes/base_link.STL" />
       </geometry>
-      <material name="powder_red">
+      <material name="">
         <color rgba="${powder_red_rgba}" />
       </material>
@@ -124,5 +125,5 @@
         <mesh filename="package://volcaniarm_description/meshes/fl_table_leg_link.STL" />
       </geometry>
-      <material name="powder_red">
+      <material name="">
         <color rgba="${powder_red_rgba}" />
       </material>
@@ -153,5 +154,5 @@
         <mesh filename="package://volcaniarm_description/meshes/fl_caster_wheel_mount_link.STL" />
       </geometry>
-      <material name="galvanized">
+      <material name="">
         <color rgba="${galvanized_rgba}" />
       </material>
@@ -182,5 +183,5 @@
         <mesh filename="package://volcaniarm_description/meshes/fl_caster_wheel_link.STL" />
       </geometry>
-      <material name="galvanized">
+      <material name="">
         <color rgba="${galvanized_rgba}" />
       </material>
@@ -211,5 +212,5 @@
         <mesh filename="package://volcaniarm_description/meshes/fr_table_leg_link.STL" />
       </geometry>
-      <material name="powder_red">
+      <material name="">
         <color rgba="${powder_red_rgba}" />
       </material>
@@ -240,5 +241,5 @@
         <mesh filename="package://volcaniarm_description/meshes/fr_caster_wheel_mount_link.STL" />
       </geometry>
-      <material name="galvanized">
+      <material name="">
         <color rgba="${galvanized_rgba}" />
       </material>
@@ -269,5 +270,5 @@
         <mesh filename="package://volcaniarm_description/meshes/fr_caster_wheel_link.STL" />
       </geometry>
-      <material name="galvanized">
+      <material name="">
         <color rgba="${galvanized_rgba}" />
       </material>
@@ -298,5 +299,5 @@
         <mesh filename="package://volcaniarm_description/meshes/rl_table_leg_link.STL" />
       </geometry>
-      <material name="powder_red">
+      <material name="">
         <color rgba="${powder_red_rgba}" />
       </material>
@@ -327,5 +328,5 @@
         <mesh filename="package://volcaniarm_description/meshes/rl_caster_wheel_mount_link.STL" />
       </geometry>
-      <material name="galvanized">
+      <material name="">
         <color rgba="${galvanized_rgba}" />
       </material>
@@ -356,5 +357,5 @@
         <mesh filename="package://volcaniarm_description/meshes/rl_caster_wheel_link.STL" />
       </geometry>
-      <material name="galvanized">
+      <material name="">
         <color rgba="${galvanized_rgba}" />
       </material>
@@ -385,5 +386,5 @@
         <mesh filename="package://volcaniarm_description/meshes/rr_table_leg_link.STL" />
       </geometry>
-      <material name="powder_red">
+      <material name="">
         <color rgba="${powder_red_rgba}" />
       </material>
@@ -414,5 +415,5 @@
         <mesh filename="package://volcaniarm_description/meshes/rr_caster_wheel_mount_link.STL" />
       </geometry>
-      <material name="galvanized">
+      <material name="">
         <color rgba="${galvanized_rgba}" />
       </material>
@@ -443,5 +444,5 @@
         <mesh filename="package://volcaniarm_description/meshes/rr_caster_wheel_link.STL" />
       </geometry>
-      <material name="galvanized">
+      <material name="">
         <color rgba="${galvanized_rgba}" />
       </material>
@@ -472,5 +473,5 @@
         <mesh filename="package://volcaniarm_description/meshes/volcaniarm_base_link.STL" />
       </geometry>
-      <material name="steel_black">
+      <material name="">
         <color rgba="${steel_black_rgba}" />
       </material>
@@ -501,5 +502,5 @@
         <mesh filename="package://volcaniarm_description/meshes/volcaniarm_left_elbow_link.STL" />
       </geometry>
-      <material name="galvanized">
+      <material name="">
         <color rgba="${galvanized_rgba}" />
       </material>
@@ -532,5 +533,5 @@
         <mesh filename="package://volcaniarm_description/meshes/volcaniarm_left_arm_link.STL" />
       </geometry>
-      <material name="galvanized">
+      <material name="">
         <color rgba="${galvanized_rgba}" />
       </material>
@@ -564,5 +565,5 @@
         <mesh filename="package://volcaniarm_description/meshes/volcaniarm_right_elbow_link.STL" />
       </geometry>
-      <material name="galvanized">
+      <material name="">
         <color rgba="${galvanized_rgba}" />
       </material>
@@ -595,5 +596,5 @@
         <mesh filename="package://volcaniarm_description/meshes/volcaniarm_right_arm_link.STL" />
       </geometry>
-      <material name="galvanized">
+      <material name="">
         <color rgba="${galvanized_rgba}" />
       </material>
@@ -633,5 +634,5 @@
         <mesh filename="package://volcaniarm_description/meshes/camera_mount_linear_link.STL" />
       </geometry>
-      <material name="galvanized">
+      <material name="">
         <color rgba="${galvanized_rgba}" />
       </material>
@@ -661,5 +662,5 @@
         <mesh filename="package://volcaniarm_description/meshes/camera_mount_rev_link.STL" />
       </geometry>
-      <material name="plastic_black">
+      <material name="">
         <color rgba="${plastic_black_rgba}" />
       </material>
@@ -692,5 +693,5 @@
         <mesh filename="package://volcaniarm_description/meshes/camera_link.STL" />
       </geometry>
-      <material name="galvanized">
+      <material name="">
         <color rgba="${galvanized_rgba}" />
       </material>
