Commit message: Edit end effector box size in urdf file

File: src/volcaniarm_description/urdf/volcaniarm.xacro (robot description, xacro)
@@ -180,7 +180,7 @@
     <link name="end_effector_link">
         <visual>
-            <origin xyz="0 0 0" rpy="0 0 0"/>
-            <geometry>
-                <box size="0.1 0.25 0.02"/>
+            <origin xyz="-0.05 0 0" rpy="0 0 0"/>
+            <geometry>
+                <box size="0.1 0.05 0.02"/>
             </geometry>
             <material name="blue">
@@ -200,13 +200,11 @@
     </link>
     <!-- Connect end effector to forearm 1 -->
-    <joint name="end_effector_joint_1" type="revolute">
+    <joint name="end_effector_joint_1" type="fixed">
         <parent link="forearm_1_link"/>
         <child link="end_effector_link"/>
         <origin xyz="0 0 -0.3" rpy="0 0 0"/>
-        <axis xyz="0 1 0"/>
-        <limit lower="-1.57" upper="1.57" effort="50" velocity="2.0"/>
-    </joint>
-    <!-- Closing link for the second connection -->
-    <link name="closing_link">
+    </joint>
+    <!-- Virtual connection point for the second forearm -->
+    <link name="virtual_connection_link">
         <visual>
             <origin xyz="0 0 0" rpy="0 0 0"/>
@@ -223,18 +221,60 @@
         </inertial>
     </link>
-    <!-- Connect forearm 2 to closing link -->
-    <joint name="forearm_2_closing_joint" type="revolute">
+    <!-- Connect forearm 2 to virtual connection -->
+    <joint name="forearm_2_virtual_joint" type="fixed">
         <parent link="forearm_2_link"/>
-        <child link="closing_link"/>
-        <origin xyz="0 0 -0.3" rpy="0 0 0"/>
-        <axis xyz="0 1 0"/>
-        <limit lower="-1.57" upper="1.57" effort="50" velocity="2.0"/>
-    </joint>
+        <child link="virtual_connection_link"/>
+        <origin xyz="0 0 -0.3" rpy="0 0 0"/>
+    </joint>
+    <!-- Gazebo material configurations -->
+    <gazebo>
+        <plugin filename="gz-sim-joint-state-publisher-system" name="gz::sim::systems::JointStatePublisher">
+        </plugin>
+    </gazebo>
+    <!-- Apply Joint Force System for manual control -->
+    <gazebo>
+        <plugin filename="gz-sim-apply-joint-force-system" name="gz::sim::systems::ApplyJointForce">
+            <joint_name>linear_rail_joint</joint_name>
+        </plugin>
+    </gazebo>
+    <gazebo>
+        <plugin filename="gz-sim-apply-joint-force-system" name="gz::sim::systems::ApplyJointForce">
+            <joint_name>upper_arm_1_joint</joint_name>
+        </plugin>
+    </gazebo>
+    <gazebo>
+        <plugin filename="gz-sim-apply-joint-force-system" name="gz::sim::systems::ApplyJointForce">
+            <joint_name>upper_arm_2_joint</joint_name>
+        </plugin>
+    </gazebo>
+    <gazebo reference="base_link">
+        <material>Gazebo/Blue</material>
+    </gazebo>
+    <gazebo reference="linear_rail_link">
+        <material>Gazebo/Green</material>
+    </gazebo>
+    <gazebo reference="upper_arm_1_link">
+        <material>Gazebo/Blue</material>
+    </gazebo>
+    <gazebo reference="upper_arm_2_link">
+        <material>Gazebo/Blue</material>
+    </gazebo>
+    <gazebo reference="forearm_1_link">
+        <material>Gazebo/Green</material>
+    </gazebo>
+    <gazebo reference="forearm_2_link">
+        <material>Gazebo/Green</material>
+    </gazebo>
+    <gazebo reference="end_effector_link">
+        <material>Gazebo/Blue</material>
+    </gazebo>
+    <gazebo reference="virtual_connection_link">
+        <material>Gazebo/Red</material>
+    </gazebo>
     <!-- Gazebo detachable joint to close the loop -->
     <gazebo>
         <plugin filename="gz-sim-detachable-joint-system" name="gz::sim::systems::DetachableJoint">
-            <parent_link>end_effector_link</parent_link>
-            <child_model>volcaniarm</child_model>
-            <child_link>closing_link</child_link>
+            <parent_link>virtual_connection_link</parent_link>
+            <child_link>end_effector_link</child_link>
             <joint_type>fixed</joint_type>
             <initial_attached>true</initial_attached>

Commit message: Add sw2urdf meshes and urdf files

File: src/volcaniarm_description/urdf/volcaniarm.xacro (robot description, xacro)
@@ -1,284 +1,190 @@
 <?xml version="1.0"?>
-<robot xmlns:xacro="http://ros.org/wiki/xacro" name="volcaniarm">
-    <xacro:include filename="./materials.xacro"/>
-    <!-- World link for fixing the robot -->
-    <link name="world"/>
-    <!-- Fix base to world -->
-    <joint name="world_to_base" type="fixed">
-        <parent link="world"/>
-        <child link="base_link"/>
-        <origin xyz="0 0 0" rpy="0 0 0"/>
-    </joint>
-    <link name="base_link">
-        <visual>
-            <origin xyz="0 0 1.3" rpy="0 0 0"/>
-            <geometry>
-                <box size="0.7 0.3 0.1"/>
-            </geometry>
-            <material name="blue">
-            </material>
-        </visual>
-        <collision>
-            <origin xyz="0 0 1.3" rpy="0 0 0"/>
-            <geometry>
-                <box size="0.7 0.3 0.1"/>
-            </geometry>
-        </collision>
-        <inertial>
-            <origin xyz="0 0 1.3" rpy="0 0 0"/>
-            <mass value="10.0"/>
-            <inertia ixx="0.1" ixy="0.0" ixz="0.0" iyy="0.5" iyz="0.0" izz="0.5"/>
-        </inertial>
-    </link>
-    <!-- Linear rail link -->
-    <link name="linear_rail_link">
-        <visual>
-            <origin xyz="0 0 0" rpy="0 0 0"/>
-            <geometry>
-                <box size="0.1 0.25 0.05"/>
-            </geometry>
-            <material name="green">
-            </material>
-        </visual>
-        <collision>
-            <origin xyz="0 0 0" rpy="0 0 0"/>
-            <geometry>
-                <box size="0.1 0.25 0.05"/>
-            </geometry>
-        </collision>
-        <inertial>
-            <origin xyz="0 0 0" rpy="0 0 0"/>
-            <mass value="1.0"/>
-            <inertia ixx="0.01" ixy="0.0" ixz="0.0" iyy="0.01" iyz="0.0" izz="0.01"/>
-        </inertial>
-    </link>
-    <!-- Prismatic joint for linear movement -->
-    <joint name="linear_rail_joint" type="prismatic">
-        <parent link="base_link"/>
-        <child link="linear_rail_link"/>
-        <origin xyz="0 0 1.25" rpy="0 0 0"/>
-        <axis xyz="1 0 0"/>
-        <limit lower="-0.28" upper="0.28" effort="100" velocity="0.1"/>
-    </joint>
-    <!-- Upper arm 1 -->
-    <link name="upper_arm_1_link">
-        <visual>
-            <origin xyz="0 0 -0.15" rpy="0 0 0"/>
-            <geometry>
-                <cylinder radius="0.02" length="0.3"/>
-            </geometry>
-            <material name="blue">
-            </material>
-        </visual>
-        <collision>
-            <origin xyz="0 0 -0.15" rpy="0 0 0"/>
-            <geometry>
-                <cylinder radius="0.02" length="0.3"/>
-            </geometry>
-        </collision>
-        <inertial>
-            <origin xyz="0 0 -0.15" rpy="0 0 0"/>
-            <mass value="0.5"/>
-            <inertia ixx="0.004" ixy="0.0" ixz="0.0" iyy="0.004" iyz="0.0" izz="0.0001"/>
-        </inertial>
-    </link>
-    <joint name="upper_arm_1_joint" type="revolute">
-        <parent link="linear_rail_link"/>
-        <child link="upper_arm_1_link"/>
-        <origin xyz="0 0.125 0" rpy="0 0 1.57"/>
-        <axis xyz="0 1 0"/>
-        <limit lower="-1.57" upper="1.57" effort="50" velocity="2.0"/>
-    </joint>
-    <!-- Upper arm 2 -->
-    <link name="upper_arm_2_link">
-        <visual>
-            <origin xyz="0 0 -0.15" rpy="0 0 0"/>
-            <geometry>
-                <cylinder radius="0.02" length="0.3"/>
-            </geometry>
-            <material name="blue">
-            </material>
-        </visual>
-        <collision>
-            <origin xyz="0 0 -0.15" rpy="0 0 0"/>
-            <geometry>
-                <cylinder radius="0.02" length="0.3"/>
-            </geometry>
-        </collision>
-        <inertial>
-            <origin xyz="0 0 -0.15" rpy="0 0 0"/>
-            <mass value="0.5"/>
-            <inertia ixx="0.004" ixy="0.0" ixz="0.0" iyy="0.004" iyz="0.0" izz="0.0001"/>
-        </inertial>
-    </link>
-    <joint name="upper_arm_2_joint" type="revolute">
-        <parent link="linear_rail_link"/>
-        <child link="upper_arm_2_link"/>
-        <origin xyz="0 -0.125 0" rpy="0 0 1.57"/>
-        <axis xyz="0 1 0"/>
-        <limit lower="-1.57" upper="1.57" effort="50" velocity="2.0"/>
-    </joint>
-    <!-- Forearm 1 -->
-    <link name="forearm_1_link">
-        <visual>
-            <origin xyz="0 0 -0.15" rpy="0 0 0"/>
-            <geometry>
-                <cylinder radius="0.015" length="0.3"/>
-            </geometry>
-            <material name="green">
-            </material>
-        </visual>
-        <collision>
-            <origin xyz="0 0 -0.15" rpy="0 0 0"/>
-            <geometry>
-                <cylinder radius="0.015" length="0.3"/>
-            </geometry>
-        </collision>
-        <inertial>
-            <origin xyz="0 0 -0.15" rpy="0 0 0"/>
-            <mass value="0.3"/>
-            <inertia ixx="0.002" ixy="0.0" ixz="0.0" iyy="0.002" iyz="0.0" izz="0.00007"/>
-        </inertial>
-    </link>
-    <joint name="forearm_1_joint" type="revolute">
-        <parent link="upper_arm_1_link"/>
-        <child link="forearm_1_link"/>
-        <origin xyz="0 0 -0.3" rpy="0 0 0"/>
-        <axis xyz="0 1 0"/>
-        <limit lower="-1.57" upper="1.57" effort="50" velocity="2.0"/>
-    </joint>
-    <!-- Forearm 2 -->
-    <link name="forearm_2_link">
-        <visual>
-            <origin xyz="0 0 -0.15" rpy="0 0 0"/>
-            <geometry>
-                <cylinder radius="0.015" length="0.3"/>
-            </geometry>
-            <material name="green">
-            </material>
-        </visual>
-        <collision>
-            <origin xyz="0 0 -0.15" rpy="0 0 0"/>
-            <geometry>
-                <cylinder radius="0.015" length="0.3"/>
-            </geometry>
-        </collision>
-        <inertial>
-            <origin xyz="0 0 -0.15" rpy="0 0 0"/>
-            <mass value="0.3"/>
-            <inertia ixx="0.002" ixy="0.0" ixz="0.0" iyy="0.002" iyz="0.0" izz="0.00007"/>
-        </inertial>
-    </link>
-    <joint name="forearm_2_joint" type="revolute">
-        <parent link="upper_arm_2_link"/>
-        <child link="forearm_2_link"/>
-        <origin xyz="0 0 -0.3" rpy="0 0 0"/>
-        <axis xyz="0 1 0"/>
-        <limit lower="-1.57" upper="1.57" effort="50" velocity="2.0"/>
-    </joint>
-    <!-- End effector platform -->
-    <link name="end_effector_link">
-        <visual>
-            <origin xyz="-0.05 0 0" rpy="0 0 0"/>
-            <geometry>
-                <box size="0.1 0.05 0.02"/>
-            </geometry>
-            <material name="blue">
-            </material>
-        </visual>
-        <collision>
-            <origin xyz="0 0 0" rpy="0 0 0"/>
-            <geometry>
-                <box size="0.08 0.23 0.015"/>
-            </geometry>
-        </collision>
-        <inertial>
-            <origin xyz="0 0 0" rpy="0 0 0"/>
-            <mass value="0.1"/>
-            <inertia ixx="0.0001" ixy="0.0" ixz="0.0" iyy="0.0001" iyz="0.0" izz="0.0001"/>
-        </inertial>
-    </link>
-    <!-- Connect end effector to forearm 1 -->
-    <joint name="end_effector_joint_1" type="fixed">
-        <parent link="forearm_1_link"/>
-        <child link="end_effector_link"/>
-        <origin xyz="0 0 -0.3" rpy="0 0 0"/>
-    </joint>
-    <!-- Virtual connection point for the second forearm -->
-    <link name="virtual_connection_link">
-        <visual>
-            <origin xyz="0 0 0" rpy="0 0 0"/>
-            <geometry>
-                <sphere radius="0.005"/>
-            </geometry>
-            <material name="red">
-            </material>
-        </visual>
-        <inertial>
-            <origin xyz="0 0 0" rpy="0 0 0"/>
-            <mass value="0.001"/>
-            <inertia ixx="0.000001" ixy="0.0" ixz="0.0" iyy="0.000001" iyz="0.0" izz="0.000001"/>
-        </inertial>
-    </link>
-    <!-- Connect forearm 2 to virtual connection -->
-    <joint name="forearm_2_virtual_joint" type="fixed">
-        <parent link="forearm_2_link"/>
-        <child link="virtual_connection_link"/>
-        <origin xyz="0 0 -0.3" rpy="0 0 0"/>
-    </joint>
-    <!-- Gazebo material configurations -->
-    <gazebo>
-        <plugin filename="gz-sim-joint-state-publisher-system" name="gz::sim::systems::JointStatePublisher">
-        </plugin>
-    </gazebo>
-    <!-- Apply Joint Force System for manual control -->
-    <gazebo>
-        <plugin filename="gz-sim-apply-joint-force-system" name="gz::sim::systems::ApplyJointForce">
-            <joint_name>linear_rail_joint</joint_name>
-        </plugin>
-    </gazebo>
-    <gazebo>
-        <plugin filename="gz-sim-apply-joint-force-system" name="gz::sim::systems::ApplyJointForce">
-            <joint_name>upper_arm_1_joint</joint_name>
-        </plugin>
-    </gazebo>
-    <gazebo>
-        <plugin filename="gz-sim-apply-joint-force-system" name="gz::sim::systems::ApplyJointForce">
-            <joint_name>upper_arm_2_joint</joint_name>
-        </plugin>
-    </gazebo>
-    <gazebo reference="base_link">
-        <material>Gazebo/Blue</material>
-    </gazebo>
-    <gazebo reference="linear_rail_link">
-        <material>Gazebo/Green</material>
-    </gazebo>
-    <gazebo reference="upper_arm_1_link">
-        <material>Gazebo/Blue</material>
-    </gazebo>
-    <gazebo reference="upper_arm_2_link">
-        <material>Gazebo/Blue</material>
-    </gazebo>
-    <gazebo reference="forearm_1_link">
-        <material>Gazebo/Green</material>
-    </gazebo>
-    <gazebo reference="forearm_2_link">
-        <material>Gazebo/Green</material>
-    </gazebo>
-    <gazebo reference="end_effector_link">
-        <material>Gazebo/Blue</material>
-    </gazebo>
-    <gazebo reference="virtual_connection_link">
-        <material>Gazebo/Red</material>
-    </gazebo>
-    <!-- Gazebo detachable joint to close the loop -->
-    <gazebo>
-        <plugin filename="gz-sim-detachable-joint-system" name="gz::sim::systems::DetachableJoint">
-            <parent_link>virtual_connection_link</parent_link>
-            <child_link>end_effector_link</child_link>
-            <joint_type>fixed</joint_type>
-            <initial_attached>true</initial_attached>
-            <suppress_child_warning>true</suppress_child_warning>
-        </plugin>
-    </gazebo>
+<robot xmlns:xacro="http://www.ros.org/wiki/xacro" name="volcaniarm">
+  <!-- World link (fixed reference frame) -->
+  <link name="world"/>
+  <!-- Fixed joint to keep the robot in place -->
+  <joint name="world_to_base" type="fixed">
+    <origin xyz="0 0 1.0" rpy="0 0 0"/>
+    <parent link="world"/>
+    <child link="volcaniarm_base_link"/>
+  </joint>
+  <!-- volcaniarm_base_link -->
+  <link name="volcaniarm_base_link">
+    <inertial>
+      <origin xyz="-0.0270292275136268 0.0131760845218784 -0.0373225307756109" rpy="0 0 0"/>
+      <mass value="13.6269163204302"/>
+      <inertia ixx="0.0576447761387568" ixy="2.74831669755734E-05" ixz="5.43946096689231E-06"
+               iyy="1.21122548907616" iyz="-1.83402806932084E-05" izz="1.26082925995101"/>
+    </inertial>
+    <visual>
+      <origin xyz="0 0 0" rpy="0 0 0"/>
+      <geometry>
+        <mesh filename="package://volcaniarm_description/meshes/volcaniarm_base_link.STL"/>
+      </geometry>
+      <material name="">
+        <color rgba="0.792156862745098 0.819607843137255 0.933333333333333 1"/>
+      </material>
+    </visual>
+    <collision>
+      <origin xyz="0 0 0" rpy="0 0 0"/>
+      <geometry>
+        <mesh filename="package://volcaniarm_description/meshes/volcaniarm_base_link.STL"/>
+      </geometry>
+    </collision>
+  </link>
+  <!-- delta_arm_base_link -->
+  <link name="delta_arm_base_link">
+    <inertial>
+      <origin xyz="-0.00902773080675034 -1.78293986968781E-05 -0.0512376164000921" rpy="0 0 0"/>
+      <mass value="2.15013589886699"/>
+      <inertia ixx="0.00670575094115183" ixy="-5.65872149932825E-09" ixz="2.35502761390986E-06"
+               iyy="0.00584240556923599" iyz="3.00404195469226E-11" izz="0.0113637883201367"/>
+    </inertial>
+    <visual>
+      <origin xyz="0 0 0" rpy="0 0 0"/>
+      <geometry>
+        <mesh filename="package://volcaniarm_description/meshes/delta_arm_base_link.STL"/>
+      </geometry>
+      <material name="">
+        <color rgba="0.792156862745098 0.819607843137255 0.933333333333333 1"/>
+      </material>
+    </visual>
+    <collision>
+      <origin xyz="0 0 0" rpy="0 0 0"/>
+      <geometry>
+        <mesh filename="package://volcaniarm_description/meshes/delta_arm_base_link.STL"/>
+      </geometry>
+    </collision>
+  </link>
+  <joint name="delta_arm_base_joint" type="prismatic">
+    <origin xyz="-0.069512 0 -0.0905" rpy="0 0 0"/>
+    <parent link="volcaniarm_base_link"/>
+    <child link="delta_arm_base_link"/>
+    <axis xyz="-1 0 0"/>
+    <limit lower="-0.5" upper="0.3" effort="10" velocity="10"/>
+  </joint>
+  <!-- right_elbow_link -->
+  <link name="right_elbow_link">
+    <inertial>
+      <origin xyz="-1.10526378793718E-05 8.25561841111266E-13 0.169908181946343" rpy="0 0 0"/>
+      <mass value="0.57558402444417"/>
+      <inertia ixx="0.00641206627372397" ixy="-1.17949337905161E-19" ixz="-1.08070667288964E-06"
+               iyy="0.00641457318952708" iyz="-3.11708124589583E-19" izz="0.000156325566535823"/>
+    </inertial>
+    <visual>
+      <origin xyz="0 0 0" rpy="0 0 0"/>
+      <geometry>
+        <mesh filename="package://volcaniarm_description/meshes/right_elbow_link.STL"/>
+      </geometry>
+      <material name="">
+        <color rgba="0.792156862745098 0.819607843137255 0.933333333333333 1"/>
+      </material>
+    </visual>
+    <collision>
+      <origin xyz="0 0 0" rpy="0 0 0"/>
+      <geometry>
+        <mesh filename="package://volcaniarm_description/meshes/right_elbow_link.STL"/>
+      </geometry>
+    </collision>
+  </link>
+  <joint name="right_elbow_joint" type="revolute">
+    <origin xyz="0.03 -0.085 -0.1035" rpy="2.4621 0 0"/>
+    <parent link="delta_arm_base_link"/>
+    <child link="right_elbow_link"/>
+    <axis xyz="1 0 0"/>
+    <limit lower="-1.57" upper="1.57" effort="10" velocity="10"/>
+  </joint>
+  <!-- left_elbow_link -->
+  <link name="left_elbow_link">
+    <inertial>
+      <origin xyz="-1.10526381558174E-05 -3.52899931499451E-11 0.169908182007537" rpy="0 0 0"/>
+      <mass value="0.575584024444165"/>
+      <inertia ixx="0.00641206627372392" ixy="5.31513174401966E-20" ixz="-1.08070667288878E-06"
+               iyy="0.00641457318952703" iyz="2.59530895038718E-18" izz="0.000156325566535821"/>
+    </inertial>
+    <visual>
+      <origin xyz="0 0 0" rpy="0 0 0"/>
+      <geometry>
+        <mesh filename="package://volcaniarm_description/meshes/left_elbow_link.STL"/>
+      </geometry>
+      <material name="">
+        <color rgba="0.792156862745098 0.819607843137255 0.933333333333333 1"/>
+      </material>
+    </visual>
+    <collision>
+      <origin xyz="0 0 0" rpy="0 0 0"/>
+      <geometry>
+        <mesh filename="package://volcaniarm_description/meshes/left_elbow_link.STL"/>
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
Commit message: Add feild.sdf world file

File: src/volcaniarm_description/urdf/volcaniarm.xacro (robot description, xacro)
@@ -121,5 +121,5 @@
   </joint>
   <!-- right_arm_link -->
-  <link name="right_arm_link">
+  <!-- <link name="right_arm_link">
     <inertial>
       <origin xyz="-0.00171452755479162 1.13797860024079E-12 0.23102414279737" rpy="0 0 0"/>
@@ -148,7 +148,7 @@
     <axis xyz="-1 0 0"/>
     <limit lower="-1.57" upper="1.57" effort="10" velocity="10"/>
-  </joint>
+  </joint> -->
   <!-- left_arm_link -->
-  <link name="left_arm_link">
+  <!-- <link name="left_arm_link">
     <inertial>
       <origin xyz="0.0017145275657231 2.87547763377916E-13 0.231024142798437" rpy="0 0 0"/>
@@ -177,4 +177,4 @@
     <axis xyz="1 0 0"/>
     <limit lower="-1.57" upper="1.57" effort="0" velocity="0"/>
-  </joint>
+  </joint> -->
 </robot>

Commit message: Add depth camera plugin

File: src/volcaniarm_description/urdf/volcaniarm.xacro (robot description, xacro)
@@ -1,6 +1,8 @@
 <?xml version="1.0"?>
 <robot xmlns:xacro="http://www.ros.org/wiki/xacro" name="volcaniarm">
+  <xacro:arg name="is_ignition" default="true" />
   <!-- Include materials -->
   <xacro:include filename="$(find volcaniarm_description)/urdf/materials.xacro"/>
+  <xacro:include filename="$(find volcaniarm_description)/urdf/volcaniarm_gazebo.xacro"/>
   <!-- World link (fixed reference frame) -->
   <link name="world"/>
@@ -178,3 +180,44 @@
     <limit lower="-1.57" upper="1.57" effort="0" velocity="0"/>
   </joint> -->
+  <!-- Depth Camera -->
+  <joint type="fixed" name="camera_joint">
+    <origin xyz="0.6 0 0.07" rpy="0 0.2 0"/>
+    <child link="camera_link"/>
+    <parent link="volcaniarm_base_link"/>
+    <axis xyz="0 1 0" />
+  </joint>
+  <link name='camera_link'>
+    <pose>0 0 0 0 0 0</pose>
+    <inertial>
+      <mass value="0.1"/>
+      <origin xyz="0 0 0" rpy="0 0 0"/>
+      <inertia
+          ixx="1e-6" ixy="0" ixz="0"
+          iyy="1e-6" iyz="0"
+          izz="1e-6"
+      />
+    </inertial>
+    <collision name='collision'>
+      <origin xyz="0 0 0" rpy="0 0 0"/>
+      <geometry>
+         <box size=".03 .03 .03"/>
+      </geometry>
+    </collision>
+    <visual name='camera_link_visual'>
+      <origin xyz="0 0 0" rpy="0 0 0"/>
+      <geometry>
+        <box size=".03 .03 .03"/>
+      </geometry>
+    </visual>
+  </link>
+  <gazebo reference="camera_link">
+    <material>Gazebo/Red</material>
+  </gazebo>
+  <joint type="fixed" name="camera_optical_joint">
+    <origin xyz="0 0 0" rpy="-1.5707 0 -1.5707"/>
+    <child link="camera_link_optical"/>
+    <parent link="camera_link"/>
+  </joint>
+  <link name="camera_link_optical">
+  </link>
 </robot>
