Commit message: Add basic arm controller

File: src/volcaniarm_description/urdf/volcaniarm.xacro (robot description, xacro)
@@ -5,4 +5,5 @@
   <xacro:include filename="$(find volcaniarm_description)/urdf/materials.xacro"/>
   <xacro:include filename="$(find volcaniarm_description)/urdf/volcaniarm_gazebo.xacro"/>
+  <xacro:include filename="$(find volcaniarm_description)/urdf/volcaniarm_ros2_control.xacro"/>
   <!-- World link (fixed reference frame) -->
   <link name="world"/>
@@ -120,5 +121,5 @@
     <child link="left_elbow_link"/>
     <axis xyz="1 0 0"/>
-    <limit lower="-1.57" upper="1.57" effort="0" velocity="0"/>
+    <limit lower="-1.57" upper="1.57" effort="10" velocity="10"/>
   </joint>
   <!-- right_arm_link -->

File: src/volcaniarm_description/urdf/volcaniarm_gazebo.xacro (robot description, xacro)
@@ -2,18 +2,18 @@
 <robot xmlns:xacro="http://www.ros.org/wiki/xacro" name="volcaniarm">
   <!-- ROS 2 Control -->
-  <!-- <gazebo> -->
+  <gazebo>
     <!-- ROS 2 Humble -->
-        <!-- <xacro:if value="$(arg is_ignition)">
+        <xacro:if value="$(arg is_ignition)">
             <plugin filename="ign_ros2_control-system" name="ign_ros2_control::IgnitionROS2ControlPlugin">
                 <parameters>$(find volcaniarm_controller)/config/volcaniarm_controllers.yaml</parameters>
             </plugin>
-        </xacro:if> -->
+        </xacro:if>
         <!-- ROS 2 Iron or above -->
-        <!-- <xacro:unless value="$(arg is_ignition)">
+        <xacro:unless value="$(arg is_ignition)">
             <plugin filename="gz_ros2_control-system" name="gz_ros2_control::GazeboSimROS2ControlPlugin">
                 <parameters>$(find volcaniarm_controller)/config/volcaniarm_controllers.yaml</parameters>
             </plugin>
         </xacro:unless>
-  </gazebo> -->
+  </gazebo>
     <gazebo reference="camera_link">
         <sensor name="rgbd_camera" type="rgbd_camera">

Commit message: Add end effector marker, Y-Z plane need to be fixed for the right oreintation

File: src/volcaniarm_description/urdf/volcaniarm.xacro (robot description, xacro)
@@ -63,5 +63,6 @@
     <child link="delta_arm_base_link"/>
     <axis xyz="-1 0 0"/>
-    <limit lower="-0.5" upper="0.3" effort="10" velocity="10"/>
+    <limit lower="-0.5" upper="0.3" effort="2" velocity="2"/>
+    <dynamics damping="5.0" friction="0.9"/>
   </joint>
   <!-- right_elbow_link -->

Commit message: Fix depth camera orientation

File: src/volcaniarm_description/urdf/volcaniarm.xacro (robot description, xacro)
@@ -184,5 +184,5 @@
   <!-- Depth Camera -->
   <joint type="fixed" name="camera_joint">
-    <origin xyz="0.6 0 0.07" rpy="0 0.2 0"/>
+    <origin xyz="0.65 0 -0.14" rpy="0 2.1 0"/>
     <child link="camera_link"/>
     <parent link="volcaniarm_base_link"/>

Commit message: Fix rviz config file for display.launch.py

File: src/volcaniarm_description/urdf/volcaniarm.xacro (robot description, xacro)
@@ -184,5 +184,5 @@
   <!-- Depth Camera -->
   <joint type="fixed" name="camera_joint">
-    <origin xyz="0.65 0 -0.14" rpy="0 2.1 0"/>
+    <origin xyz="0.65 0 -0.14" rpy="3.14 2.1 0"/>
     <child link="camera_link"/>
     <parent link="volcaniarm_base_link"/>
