Commit message: Bringup controller arg: traj | policy | all (runtime-switchable only in 'all')

File: src/volcaniarm_description/urdf/volcaniarm_gazebo.xacro (robot description, xacro)
@@ -2,9 +2,17 @@
 <robot xmlns:xacro="http://www.ros.org/wiki/xacro" name="volcaniarm">
   <!-- ROS 2 Control (Jazzy - Gazebo) -->
-  <!-- Both YAMLs are loaded so runtime controller switching works. -->
+  <!-- YAML(s) loaded depend on the `controller` xacro arg:
+         traj   → trajectory YAML only
+         policy → RL YAML only
+         all    → both (runtime switching enabled) -->
+  <xacro:property name="_ctrl" value="$(arg controller)" />
   <gazebo>
     <plugin filename="gz_ros2_control-system" name="gz_ros2_control::GazeboSimROS2ControlPlugin">
-      <parameters>$(find volcaniarm_controller)/config/volcaniarm_controllers.yaml</parameters>
-      <parameters>$(find volcaniarm_controller)/config/volcaniarm_rl_controller.yaml</parameters>
+      <xacro:if value="${_ctrl == 'traj' or _ctrl == 'all'}">
+        <parameters>$(find volcaniarm_controller)/config/volcaniarm_controllers.yaml</parameters>
+      </xacro:if>
+      <xacro:if value="${_ctrl == 'policy' or _ctrl == 'all'}">
+        <parameters>$(find volcaniarm_controller)/config/volcaniarm_rl_controller.yaml</parameters>
+      </xacro:if>
     </plugin>
   </gazebo>
