Commit message: Always publish RealSense color+depth frames (was real-hardware-only)
The color/depth + optical frame chain lived under <xacro:unless use_sim>,
so in sim mode (gazebo and isaac) robot_state_publisher never broadcast
camera_color_optical_frame / camera_depth_optical_frame. RViz then
couldn't transform the pointcloud or image from those frames (Isaac
publishes with frame_id=camera_color_optical_frame by RealSense
convention).

Pull the color and depth frame chains out of the unless block so they
exist in all modes. Keep camera_camera_link inside the unless block —
that's the RealSense driver's internal base, only relevant when the
driver runs alongside robot_state_publisher on real hardware.

File: src/volcaniarm_description/urdf/volcaniarm_realsense.xacro (robot description, xacro)
@@ -12,5 +12,36 @@
     </joint>
   </xacro:if>
-  <!-- Real hardware: RealSense D435i extra frames (only when not simulating) -->
+  <!-- RealSense D435i frame chain. Published by robot_state_publisher in all
+       modes so pointcloud/image frame_ids (camera_color_optical_frame etc.,
+       emitted by the RealSense driver on real hardware AND by Isaac's ROS2
+       bridge in sim) resolve in RViz. Harmless in Gazebo — Gazebo's rgbd
+       sensor publishes its own internal frames separately. -->
+  <link name="camera_depth_frame" />
+  <joint name="camera_depth_joint" type="fixed">
+    <origin xyz="0 0 0" rpy="0 0 0" />
+    <parent link="camera_link" />
+    <child link="camera_depth_frame" />
+  </joint>
+  <link name="camera_depth_optical_frame" />
+  <joint name="camera_depth_optical_joint" type="fixed">
+    <origin xyz="0 0 0" rpy="-1.5708 0 -1.5708" />
+    <parent link="camera_depth_frame" />
+    <child link="camera_depth_optical_frame" />
+  </joint>
+  <link name="camera_color_frame" />
+  <joint name="camera_color_joint" type="fixed">
+    <origin xyz="0 0 0" rpy="0 0 0" />
+    <parent link="camera_link" />
+    <child link="camera_color_frame" />
+  </joint>
+  <link name="camera_color_optical_frame" />
+  <joint name="camera_color_optical_joint" type="fixed">
+    <origin xyz="0 0 0" rpy="-1.5708 0 -1.5708" />
+    <parent link="camera_color_frame" />
+    <child link="camera_color_optical_frame" />
+  </joint>
+  <!-- Real hardware only: extra camera_camera_link (the RealSense driver's
+       internal base), inserted between camera_link and the driver-published
+       frames when the driver runs alongside robot_state_publisher. -->
   <xacro:unless value="$(arg use_sim)">
     <link name="camera_camera_link" />
@@ -20,28 +51,4 @@
       <child link="camera_camera_link" />
     </joint>
-    <link name="camera_depth_frame" />
-    <joint name="camera_depth_joint" type="fixed">
-      <origin xyz="0 0 0" rpy="0 0 0" />
-      <parent link="camera_camera_link" />
-      <child link="camera_depth_frame" />
-    </joint>
-    <link name="camera_depth_optical_frame" />
-    <joint name="camera_depth_optical_joint" type="fixed">
-      <origin xyz="0 0 0" rpy="-1.5708 0 -1.5708" />
-      <parent link="camera_depth_frame" />
-      <child link="camera_depth_optical_frame" />
-    </joint>
-    <link name="camera_color_frame" />
-    <joint name="camera_color_joint" type="fixed">
-      <origin xyz="0 0 0" rpy="0 0 0" />
-      <parent link="camera_camera_link" />
-      <child link="camera_color_frame" />
-    </joint>
-    <link name="camera_color_optical_frame" />
-    <joint name="camera_color_optical_joint" type="fixed">
-      <origin xyz="0 0 0" rpy="-1.5708 0 -1.5708" />
-      <parent link="camera_color_frame" />
-      <child link="camera_color_optical_frame" />
-    </joint>
   </xacro:unless>
 </robot>

Commit message: Always expose RealSense optical frames (sim too, so Isaac TF resolves)

File: src/volcaniarm_description/urdf/volcaniarm_realsense.xacro (robot description, xacro)
@@ -12,36 +12,38 @@
     </joint>
   </xacro:if>
-  <!-- Real hardware: RealSense D435i extra frames (only when not simulating) -->
-  <xacro:unless value="$(arg use_sim)">
-    <link name="camera_camera_link" />
-    <joint name="camera_to_realsense" type="fixed">
-      <origin xyz="0 0 0" rpy="0 0 0" />
-      <parent link="camera_link" />
-      <child link="camera_camera_link" />
-    </joint>
-    <link name="camera_depth_frame" />
-    <joint name="camera_depth_joint" type="fixed">
-      <origin xyz="0 0 0" rpy="0 0 0" />
-      <parent link="camera_camera_link" />
-      <child link="camera_depth_frame" />
-    </joint>
-    <link name="camera_depth_optical_frame" />
-    <joint name="camera_depth_optical_joint" type="fixed">
-      <origin xyz="0 0 0" rpy="-1.5708 0 -1.5708" />
-      <parent link="camera_depth_frame" />
-      <child link="camera_depth_optical_frame" />
-    </joint>
-    <link name="camera_color_frame" />
-    <joint name="camera_color_joint" type="fixed">
-      <origin xyz="0 0 0" rpy="0 0 0" />
-      <parent link="camera_camera_link" />
-      <child link="camera_color_frame" />
-    </joint>
-    <link name="camera_color_optical_frame" />
-    <joint name="camera_color_optical_joint" type="fixed">
-      <origin xyz="0 0 0" rpy="-1.5708 0 -1.5708" />
-      <parent link="camera_color_frame" />
-      <child link="camera_color_optical_frame" />
-    </joint>
-  </xacro:unless>
+  <!-- RealSense D435i extra frames. Defined in every mode (real and sim)
+       so that topics published with `frame_id=camera_color_optical_frame`
+       or `camera_depth_optical_frame` — by the real camera driver, by
+       Isaac Sim's ROS2 graph, or by Gazebo's sensor plugin — resolve in
+       TF. Harmless to have in Gazebo: no visuals/collisions/inertials. -->
+  <link name="camera_camera_link" />
+  <joint name="camera_to_realsense" type="fixed">
+    <origin xyz="0 0 0" rpy="0 0 0" />
+    <parent link="camera_link" />
+    <child link="camera_camera_link" />
+  </joint>
+  <link name="camera_depth_frame" />
+  <joint name="camera_depth_joint" type="fixed">
+    <origin xyz="0 0 0" rpy="0 0 0" />
+    <parent link="camera_camera_link" />
+    <child link="camera_depth_frame" />
+  </joint>
+  <link name="camera_depth_optical_frame" />
+  <joint name="camera_depth_optical_joint" type="fixed">
+    <origin xyz="0 0 0" rpy="-1.5708 0 -1.5708" />
+    <parent link="camera_depth_frame" />
+    <child link="camera_depth_optical_frame" />
+  </joint>
+  <link name="camera_color_frame" />
+  <joint name="camera_color_joint" type="fixed">
+    <origin xyz="0 0 0" rpy="0 0 0" />
+    <parent link="camera_camera_link" />
+    <child link="camera_color_frame" />
+  </joint>
+  <link name="camera_color_optical_frame" />
+  <joint name="camera_color_optical_joint" type="fixed">
+    <origin xyz="0 0 0" rpy="-1.5708 0 -1.5708" />
+    <parent link="camera_color_frame" />
+    <child link="camera_color_optical_frame" />
+  </joint>
 </robot>

Commit message: Pull calibration camera further along base_link +X to fit both tags
Camera was at base_link xyz=(0.8, 0, -0.68) -> world (-0.8, 0, 0.30),
which framed the EE but the base tag fell out of view. Pull it to
xyz=(1.5, 0, -0.48) -> world (-1.5, 0, 0.5): farther back so the
vertical FOV covers both the base tag and the arm's home pose, and
slightly higher to roughly center on the workspace. Comment in the
xacro updated to match.

File: src/volcaniarm_description/urdf/volcaniarm_realsense.xacro (robot description, xacro)
@@ -3,9 +3,10 @@
   <!-- Calibration mode: camera at fixed position in front of robot (sim only).
        base_link is at world (0,0,0.98) with yaw=pi, so base_link +X = world -X.
-       Camera at world (-1.5, 0, 0.5) facing world +X (toward robot):
-         In base_link frame: xyz=(1.5, 0, -0.48), yaw=pi to face base_link -X = world +X. -->
+       Camera pulled out far enough in base_link +X to fit both the base
+       and EE AprilTags in the same frame; height tuned to roughly center
+       on the arm's reachable workspace. -->
   <xacro:if value="$(arg calibration)">
     <joint name="calibration_camera_joint" type="fixed">
-      <origin xyz="0.8 0 -0.68" rpy="0 0 ${pi}" />
+      <origin xyz="1.5 0 -0.48" rpy="0 0 ${pi}" />
       <parent link="base_link" />
       <child link="camera_link" />

Commit message: Pull calibration camera further back to fully fit base tag
Camera was at base_link X=1.5 (world X=-1.5); base tag was clipping
at the bottom of the frame. Bump X to 2.0 (world X=-2.0) so the
vertical FOV at base-tag distance widens by ~30% and the tag sits
fully inside the image.

File: src/volcaniarm_description/urdf/volcaniarm_realsense.xacro (robot description, xacro)
@@ -8,5 +8,5 @@
   <xacro:if value="$(arg calibration)">
     <joint name="calibration_camera_joint" type="fixed">
-      <origin xyz="1.5 0 -0.48" rpy="0 0 ${pi}" />
+      <origin xyz="2.0 0 -0.48" rpy="0 0 ${pi}" />
       <parent link="base_link" />
       <child link="camera_link" />

Commit message: Raise + pitch the calibration camera so the EE tag is detectable
The EE AprilTag is mounted to face world +Z (straight up) so the
original down-looking arm-mounted camera could read it. In
calibration mode we use a fixed side camera; with rpy='0 0 pi' the
optical axis was horizontal, so the camera saw the EE tag edge-on
and apriltag_ros could not detect it (the base tag, which faces
world -X, was fine).

Move the calibration camera from base_link xyz=(2.0, 0, -0.48) /
yaw=pi to xyz=(2.0, 0, 0.22) / rpy='0 0.5 pi'. World pose goes from
(-2.0, 0, 0.5) horizontal to (-2.0, 0, 1.2) tilted ~28.6 deg
downward, which puts both tag faces within the camera's vertical
FOV and at recoverable detection angles (well under apriltag's
oblique-view limit).

File: src/volcaniarm_description/urdf/volcaniarm_realsense.xacro (robot description, xacro)
@@ -3,10 +3,15 @@
   <!-- Calibration mode: camera at fixed position in front of robot (sim only).
        base_link is at world (0,0,0.98) with yaw=pi, so base_link +X = world -X.
-       Camera pulled out far enough in base_link +X to fit both the base
-       and EE AprilTags in the same frame; height tuned to roughly center
-       on the arm's reachable workspace. -->
+       Camera at world (-2.0, 0, 1.2) pitched ~28.6 deg downward so it can
+       see both AprilTag faces:
+         - EE tag normal points world +Z (up), only detectable when the
+           camera looks down at it.
+         - Base tag normal points world -X (toward the camera), still in
+           frame at this height/pitch combination.
+       In base_link frame: xyz=(2.0, 0, 0.22), rpy yaw=pi puts +X back
+       toward world +X, pitch=0.5 rad tilts the optical axis downward. -->
   <xacro:if value="$(arg calibration)">
     <joint name="calibration_camera_joint" type="fixed">
-      <origin xyz="2.0 0 -0.48" rpy="0 0 ${pi}" />
+      <origin xyz="2.0 0 0.22" rpy="0 0.5 ${pi}" />
       <parent link="base_link" />
       <child link="camera_link" />

Commit message: Restore horizontal calibration camera, document EE-edge-on caveat
Reverts the diagonal pitch tweak. Camera goes back to horizontal
viewing at world (-2.0, 0, 0.5) per the user's preference. Comment
in the xacro now flags the geometry trade-off: at home pose the EE
tag faces world +Z, so a horizontal camera sees it edge-on and
apriltag cannot decode the tag until the arm rotates. The base tag
remains detectable at home since its normal already points toward
the camera (-X).

File: src/volcaniarm_description/urdf/volcaniarm_realsense.xacro (robot description, xacro)
@@ -1,17 +1,17 @@
 <?xml version="1.0"?>
 <robot xmlns:xacro="http://www.ros.org/wiki/xacro" name="volcaniarm_realsense">
-  <!-- Calibration mode: camera at fixed position in front of robot (sim only).
-       base_link is at world (0,0,0.98) with yaw=pi, so base_link +X = world -X.
-       Camera at world (-2.0, 0, 1.2) pitched ~28.6 deg downward so it can
-       see both AprilTag faces:
-         - EE tag normal points world +Z (up), only detectable when the
-           camera looks down at it.
-         - Base tag normal points world -X (toward the camera), still in
-           frame at this height/pitch combination.
-       In base_link frame: xyz=(2.0, 0, 0.22), rpy yaw=pi puts +X back
-       toward world +X, pitch=0.5 rad tilts the optical axis downward. -->
+  <!-- Calibration mode: horizontal camera in front of the robot (sim only).
+       base_link is at world (0,0,0.98) with yaw=pi, so base_link +X is
+       world -X. xyz=(2.0, 0, -0.48) -> world (-2.0, 0, 0.5); yaw=pi
+       points +X back toward world +X. Z is set near the midpoint of the
+       EE-tag and base-tag world heights so both fit in the vertical FOV.
+       NOTE: at home (theta=0,0) the EE tag normal points world +Z, so a
+       horizontal camera sees that tag edge-on and apriltag will not
+       decode it. Detection of the EE tag becomes reliable as soon as
+       the arm starts moving. If you need home-pose EE detection, tilt
+       the camera downward or rotate the EE tag mount. -->
   <xacro:if value="$(arg calibration)">
     <joint name="calibration_camera_joint" type="fixed">
-      <origin xyz="2.0 0 0.22" rpy="0 0.5 ${pi}" />
+      <origin xyz="2.0 0 -0.48" rpy="0 0 ${pi}" />
       <parent link="base_link" />
       <child link="camera_link" />

Commit message: Edit camera position

File: src/volcaniarm_description/urdf/volcaniarm_realsense.xacro (robot description, xacro)
@@ -17,5 +17,5 @@
   <xacro:if value="$(arg calibration)">
     <joint name="calibration_camera_joint" type="fixed">
-      <origin xyz="1.8 0 -0.06" rpy="0 0 ${pi}" />
+      <origin xyz="1.8 0 -0.5" rpy="0 0 ${pi}" />
       <parent link="base_link" />
       <child link="camera_link" />

Commit message: Edit apriltag params & camera position

File: src/volcaniarm_description/urdf/volcaniarm_realsense.xacro (robot description, xacro)
@@ -17,5 +17,5 @@
   <xacro:if value="$(arg calibration)">
     <joint name="calibration_camera_joint" type="fixed">
-      <origin xyz="1.8 0 -0.5" rpy="0 0 ${pi}" />
+      <origin xyz="1.5 0 -0.5" rpy="0 0 ${pi}" />
       <parent link="base_link" />
       <child link="camera_link" />
