Commit message: Add new delta arm urdf file. ee marker need to be tuned

File: src/volcaniarm_description/urdf/volcaniarm_ros2_control.xacro (robot description, xacro)
@@ -3,29 +3,13 @@
     <ros2_control name="RobotSystem" type="system">
     <!-- ros2_control Gazebo -->
-        <!-- ROS 2 Humble -->
-        <xacro:if value="$(arg is_ignition)">
-            <hardware>
-                <plugin>ign_ros2_control/IgnitionSystem</plugin>
-            </hardware>
-        </xacro:if>
-        <!-- ROS 2 Iron or above -->
-        <xacro:unless value="$(arg is_ignition)">
-            <hardware>
-                <plugin>gz_ros2_control/GazeboSimSystem</plugin>
-            </hardware>
-        </xacro:unless>
+        <!-- ROS 2 Jazzy with Gazebo -->
+        <hardware>
+            <plugin>gz_ros2_control/GazeboSimSystem</plugin>
+        </hardware>
         <!-- ros2_control Common Interfaces -->
-        <joint name="delta_arm_base_joint">
-            <command_interface name="position">
-              <param name="min">-0.5</param>
-              <param name="max">0.3</param>
-            </command_interface>
-            <state_interface name="position" />
-            <state_interface name="velocity" />
-        </joint>
         <joint name="right_elbow_joint">
             <command_interface name="position">
-              <param name="min">-2</param>
-              <param name="max">2</param>
+              <param name="min">-2.09</param>
+              <param name="max">2.09</param>
             </command_interface>
             <state_interface name="position" />
@@ -34,6 +18,6 @@
         <joint name="left_elbow_joint">
             <command_interface name="position">
-              <param name="min">-2</param>
-              <param name="max">2</param>
+              <param name="min">-2.09</param>
+              <param name="max">2.09</param>
             </command_interface>
             <state_interface name="position" />

Commit message: Add Isaac Sim support via topic-based ros2_control
New sim:=gazebo|isaac launch arg in sim_bringup.launch.py gates
gazebo.launch.py (default) vs a new isaac.launch.py that brings up
robot_state_publisher + a standalone controller_manager.

The ros2_control xacro picks the hardware plugin from a sim_engine
arg — gz_ros2_control/GazeboSimSystem for gazebo,
joint_state_topic_hardware_interface/JointStateTopicSystem for isaac
(Jazzy's successor to PickNik's topic_based_ros2_control), reading
Isaac's raw articulation feed from /isaac_joint_states and publishing
commands on /joint_commands. Elbow joints gained an effort
state_interface — required by JointStateTopicSystem, inert elsewhere.

File: src/volcaniarm_description/urdf/volcaniarm_ros2_control.xacro (robot description, xacro)
@@ -3,9 +3,24 @@
     <!-- Argument to switch between simulation and real hardware -->
     <xacro:arg name="use_sim" default="true" />
+    <!-- Simulation engine selection: "gazebo" or "isaac" (only used when use_sim=true) -->
+    <xacro:arg name="sim_engine" default="gazebo" />
+    <xacro:property name="sim_engine" value="$(arg sim_engine)" />
     <ros2_control name="RobotSystem" type="system">
     <!-- ros2_control Hardware Selection -->
         <hardware>
             <xacro:if value="$(arg use_sim)">
-                <plugin>gz_ros2_control/GazeboSimSystem</plugin>
+                <xacro:if value="${sim_engine == 'gazebo'}">
+                    <plugin>gz_ros2_control/GazeboSimSystem</plugin>
+                </xacro:if>
+                <xacro:if value="${sim_engine == 'isaac'}">
+                    <plugin>joint_state_topic_hardware_interface/JointStateTopicSystem</plugin>
+                    <param name="joint_commands_topic">/joint_commands</param>
+                    <!-- Read from Isaac's raw 4-joint publisher, not /joint_states.
+                         This keeps /joint_states owned by joint_state_broadcaster +
+                         the custom passive-joint publisher, avoiding duplicate
+                         joint-name entries on the same topic. -->
+                    <param name="joint_states_topic">/isaac_joint_states</param>
+                    <param name="sum_wrapped_joint_states">true</param>
+                </xacro:if>
             </xacro:if>
             <xacro:unless value="$(arg use_sim)">
@@ -26,4 +41,7 @@
             </state_interface>
             <state_interface name="velocity" />
+            <!-- effort state_interface required by joint_state_topic_hardware_interface (Isaac path);
+                 harmless in Gazebo and real-hw paths where the field stays at 0. -->
+            <state_interface name="effort" />
         </joint>
         <joint name="volcaniarm_left_elbow_joint">
@@ -36,4 +54,5 @@
             </state_interface>
             <state_interface name="velocity" />
+            <state_interface name="effort" />
         </joint>
     </ros2_control>

Commit message: Match ros2_control joint order to IsaacLab URDF (left, then right)

File: src/volcaniarm_description/urdf/volcaniarm_ros2_control.xacro (robot description, xacro)
@@ -37,6 +37,14 @@
         <!-- effort is exported (zero on real HW, physics value in Isaac) so the
              URDF interface set is identical across gazebo / isaac / real and
-             the JointStateTopicSystem plugin can land Isaac's effort field. -->
-        <joint name="volcaniarm_right_elbow_joint">
+             the JointStateTopicSystem plugin can land Isaac's effort field.
+             Order: left first, then right — matches the joint declaration
+             order in the IsaacLab training URDF
+             (volcaniarm_isaaclab/assets/urdf/urdf/volcaniarm.urdf). The
+             trained policy was authored against [left, right] joint order
+             for both observation and action vectors; aligning declaration
+             order here eliminates any chance of the topic-based hardware
+             interface or controller_manager binding interfaces in a
+             different order than the policy expects. -->
+        <joint name="volcaniarm_left_elbow_joint">
             <command_interface name="position">
               <param name="min">-3.14</param>
@@ -49,5 +57,5 @@
             <state_interface name="effort" />
         </joint>
-        <joint name="volcaniarm_left_elbow_joint">
+        <joint name="volcaniarm_right_elbow_joint">
             <command_interface name="position">
               <param name="min">-3.14</param>
