Commit message: hardware interface: enforce xacro command-interface position limits in write()

File: src/volcaniarm_description/urdf/volcaniarm_ros2_control.xacro (robot description, xacro)
@@ -46,8 +46,17 @@
              interface or controller_manager binding interfaces in a
              different order than the policy expects. -->
+        <!-- min/max: software travel guard, enforced by the REAL hardware
+             interface (VolcaniArmHardware clamps in write() before rad->
+             steps). Sim plugins ignore these params (Gazebo enforces the
+             URDF <limit> instead). +-2.0 rad is the hardware backstop:
+             wider than every legitimate consumer (RL trained envelope
+             +-1.309, teleop EE box, weed-targeting IK) but inside the
+             URDF mechanical +-3.14.
+             TODO(Tamir): confirm against the physical hard stops and
+             tighten further if the mechanism allows less travel. -->
         <joint name="volcaniarm_left_elbow_joint">
             <command_interface name="position">
-              <param name="min">-3.14</param>
-              <param name="max">3.14</param>
+              <param name="min">-2.0</param>
+              <param name="max">2.0</param>
             </command_interface>
             <state_interface name="position">
@@ -59,6 +68,6 @@
         <joint name="volcaniarm_right_elbow_joint">
             <command_interface name="position">
-              <param name="min">-3.14</param>
-              <param name="max">3.14</param>
+              <param name="min">-2.0</param>
+              <param name="max">2.0</param>
             </command_interface>
             <state_interface name="position">
