Commit message: Add apriltag model to gazebo

File: src/volcaniarm_description/urdf/volcaniarm_apriltag.xacro (robot description, xacro)
@@ -2,8 +2,8 @@
 <robot xmlns:xacro="http://www.ros.org/wiki/xacro" name="volcaniarm_apriltag">
   <!-- AprilTag 36h11 ID 20 mounted on the end effector (sim only).
-       The tag is a flat 64mm square facing the camera. -->
-  <xacro:property name="tag_size" value="0.064" />
-  <xacro:property name="tag_texture_path"
-    value="$(find volcaniarm_description)/meshes/apriltag_36h11_id20.png" />
+       The tag is a flat 64mm square facing +X direction.
+       Uses a DAE mesh with baked texture so it renders in both Gazebo and RViz. -->
+  <xacro:property name="tag_mesh"
+    value="package://volcaniarm_description/models/Apriltag36_11_00020/apriltag_36h11_id20.dae" />
   <!-- Tag visual link attached to right_arm_tip_link -->
   <link name="apriltag_link">
@@ -13,14 +13,15 @@
       <inertia ixx="1e-9" ixy="0" ixz="0" iyy="1e-9" iyz="0" izz="1e-9" />
     </inertial>
-    <visual name="apriltag_visual">
+    <visual>
       <origin xyz="0 0 0" rpy="0 0 0" />
       <geometry>
-        <box size="${tag_size} ${tag_size} 0.001" />
+        <mesh filename="${tag_mesh}" />
       </geometry>
     </visual>
   </link>
   <joint name="apriltag_joint" type="fixed">
-    <!-- Tag mounted on EE tip, face pointing along X axis, rotated 45 deg -->
-    <origin xyz="0.04 0 0" rpy="0 1.5708 0.7854" />
+    <!-- Tag mounted on EE tip, offset along X, face pointing in +X direction.
+         The DAE quad face is on the Z plane, so rotate 90 deg around Y to face +X. -->
+    <origin xyz="0.04 0 0" rpy="0 ${pi/2} 0" />
     <parent link="right_arm_tip_link" />
     <child link="apriltag_link" />
@@ -29,19 +30,3 @@
     <preserveFixedJoint>true</preserveFixedJoint>
   </gazebo>
-  <!-- Apply the AprilTag texture in Gazebo -->
-  <gazebo reference="apriltag_link">
-    <visual name="apriltag_visual">
-      <material>
-        <diffuse>1 1 1 1</diffuse>
-        <specular>0 0 0 0</specular>
-        <pbr>
-          <metal>
-            <albedo_map>${tag_texture_path}</albedo_map>
-            <metalness>0.0</metalness>
-            <roughness>1.0</roughness>
-          </metal>
-        </pbr>
-      </material>
-    </visual>
-  </gazebo>
 </robot>

Commit message: Add mount link to level AprilTag parallel to ground plane
Add apriltag_mount_link between right_arm_tip_link and apriltag_link
with a counter-rotation to compensate for the EE tilt, making the
tag parallel to the ground regardless of arm pose.

File: src/volcaniarm_description/urdf/volcaniarm_apriltag.xacro (robot description, xacro)
@@ -21,9 +21,27 @@
     </visual>
   </link>
+  <!-- Intermediate link to counter-rotate the EE angle so the tag is
+       parallel to the ground plane. The EE is tilted ~45 deg around X,
+       so rotate -45 deg to level it out. -->
+  <link name="apriltag_mount_link">
+    <inertial>
+      <origin xyz="0 0 0" rpy="0 0 0" />
+      <mass value="0.001" />
+      <inertia ixx="1e-9" ixy="0" ixz="0" iyy="1e-9" iyz="0" izz="1e-9" />
+    </inertial>
+  </link>
+  <joint name="apriltag_mount_joint" type="fixed">
+    <origin xyz="0.04 0 0" rpy="${-pi/3.4} 0 0" />
+    <parent link="right_arm_tip_link" />
+    <child link="apriltag_mount_link" />
+  </joint>
+  <gazebo reference="apriltag_mount_joint">
+    <preserveFixedJoint>true</preserveFixedJoint>
+  </gazebo>
   <joint name="apriltag_joint" type="fixed">
-    <!-- Tag mounted on EE tip, offset along X, face pointing in +X direction.
+    <!-- Tag face pointing in +X direction.
          The DAE quad face is on the Z plane, so rotate 90 deg around Y to face +X. -->
-    <origin xyz="0.04 0 0" rpy="0 ${pi/2} 0" />
-    <parent link="right_arm_tip_link" />
+    <origin xyz="0 0 0" rpy="0 ${pi/2} 0" />
+    <parent link="apriltag_mount_link" />
     <child link="apriltag_link" />
   </joint>

Commit message: Scaffold calibration dashboard (URDF base tag, runner, rqt plugin)
URDF: add ID-5 base-link AprilTag in volcaniarm_apriltag.xacro alongside
the existing ID-20 EE tag. Both gated by the existing $(arg calibration)
include in volcaniarm.urdf.xacro. Tag-link/joint names renamed for
symmetry (apriltag_ee_*, apriltag_base_*).

volcaniarm_calibration:
- New runner/ subpackage: CalibrationRunner with start/approve/cancel
  surface and status/preview/progress/finished callbacks; BaseTest +
  StaticAccuracyTest + RepeatabilityTest registry; RunWriter persists
  per-run timestamped folder with samples/fk/residuals/summary CSVs
  and config.yaml.
- New rqt/ subpackage: CalibrationDashboardPlugin (qt_gui.plugin.Plugin
  subclass) + CalibrationDashboardWidget (form-based UI, runner
  signals, preview/approve/cancel handshake) + PreviewPublisher
  (MarkerArray + target_ee_link static TF).
- accuracy_test_node now a thin shim around CalibrationRunner with
  auto_approve=True; existing CLI usage unchanged.
- plugin.xml, package.xml deps (rqt_gui, rqt_gui_py, pyqt5, yaml,
  visualization_msgs), CMakeLists.txt installs.

Build green; rqt --list-plugins surfaces VolcaniarmCalibrationDashboard.

File: src/volcaniarm_description/urdf/volcaniarm_apriltag.xacro (robot description, xacro)
@@ -1,12 +1,15 @@
 <?xml version="1.0"?>
 <robot xmlns:xacro="http://www.ros.org/wiki/xacro" name="volcaniarm_apriltag">
-  <!-- AprilTag 36h11 ID 20 mounted on the end effector (sim only).
-       Uses a DAE mesh with baked texture so it renders in both Gazebo and RViz.
-       DAE has 64mm geometry, scaled up to 200mm for reliable detection in sim. -->
-  <xacro:property name="tag_mesh"
+  <!-- AprilTag 36h11 markers used for hand-eye calibration and accuracy
+       tests. Both tags use a DAE mesh with baked texture so they render
+       in Gazebo and RViz. The DAE has 64mm geometry, scaled up to 200mm
+       for reliable detection in sim. -->
+  <xacro:property name="tag_scale" value="${0.2 / 0.064}" />
+  <!-- ============================================================= -->
+  <!-- ID 20: end-effector marker (right_arm_tip_link)                -->
+  <!-- ============================================================= -->
+  <xacro:property name="ee_tag_mesh"
     value="package://volcaniarm_description/models/Apriltag36_11_00020/apriltag_36h11_id20.dae" />
-  <xacro:property name="tag_scale" value="${0.2 / 0.064}" />
-  <!-- Tag visual link attached to right_arm_tip_link -->
-  <link name="apriltag_link">
+  <link name="apriltag_ee_link">
     <inertial>
       <origin xyz="0 0 0" rpy="0 0 0" />
@@ -17,12 +20,11 @@
       <origin xyz="0 0 0" rpy="0 0 0" />
       <geometry>
-        <mesh filename="${tag_mesh}" scale="${tag_scale} ${tag_scale} ${tag_scale}" />
+        <mesh filename="${ee_tag_mesh}" scale="${tag_scale} ${tag_scale} ${tag_scale}" />
       </geometry>
     </visual>
   </link>
-  <!-- Intermediate link to counter-rotate the EE angle so the tag is
-       parallel to the ground plane. The EE is tilted ~45 deg around X,
-       so rotate -45 deg to level it out. -->
-  <link name="apriltag_mount_link">
+  <!-- Intermediate link to counter-rotate the EE so the tag is
+       parallel to the ground plane. -->
+  <link name="apriltag_ee_mount_link">
     <inertial>
       <origin xyz="0 0 0" rpy="0 0 0" />
@@ -31,20 +33,63 @@
     </inertial>
   </link>
-  <joint name="apriltag_mount_joint" type="fixed">
+  <joint name="apriltag_ee_mount_joint" type="fixed">
     <origin xyz="0.04 0 0" rpy="${-pi/3.4} 0 0" />
     <parent link="right_arm_tip_link" />
-    <child link="apriltag_mount_link" />
+    <child link="apriltag_ee_mount_link" />
   </joint>
-  <gazebo reference="apriltag_mount_joint">
+  <gazebo reference="apriltag_ee_mount_joint">
     <preserveFixedJoint>true</preserveFixedJoint>
   </gazebo>
-  <joint name="apriltag_joint" type="fixed">
-    <!-- Tag face pointing in +X direction.
-         The DAE quad face is on the Z plane, so rotate 90 deg around Y to face +X. -->
+  <joint name="apriltag_ee_joint" type="fixed">
+    <!-- Tag face pointing in +X. The DAE quad face is on the Z plane,
+         so rotate 90 deg around Y to face +X. -->
     <origin xyz="0 0 0" rpy="0 ${pi/2} 0" />
-    <parent link="apriltag_mount_link" />
-    <child link="apriltag_link" />
+    <parent link="apriltag_ee_mount_link" />
+    <child link="apriltag_ee_link" />
   </joint>
-  <gazebo reference="apriltag_joint">
+  <gazebo reference="apriltag_ee_joint">
+    <preserveFixedJoint>true</preserveFixedJoint>
+  </gazebo>
+  <!-- ============================================================= -->
+  <!-- ID 5: base-link reference marker (volcaniarm_base_link)        -->
+  <!-- ============================================================= -->
+  <xacro:property name="base_tag_mesh"
+    value="package://volcaniarm_description/models/Apriltag36_11_00005/apriltag_36h11_id05.dae" />
+  <link name="apriltag_base_link">
+    <inertial>
+      <origin xyz="0 0 0" rpy="0 0 0" />
+      <mass value="0.001" />
+      <inertia ixx="1e-9" ixy="0" ixz="0" iyy="1e-9" iyz="0" izz="1e-9" />
+    </inertial>
+    <visual>
+      <origin xyz="0 0 0" rpy="0 0 0" />
+      <geometry>
+        <mesh filename="${base_tag_mesh}" scale="${tag_scale} ${tag_scale} ${tag_scale}" />
+      </geometry>
+    </visual>
+  </link>
+  <link name="apriltag_base_mount_link">
+    <inertial>
+      <origin xyz="0 0 0" rpy="0 0 0" />
+      <mass value="0.001" />
+      <inertia ixx="1e-9" ixy="0" ixz="0" iyy="1e-9" iyz="0" izz="1e-9" />
+    </inertial>
+  </link>
+  <!-- TODO(thesis): replace with the measured mount offset once the
+       printed bracket is fitted on volcaniarm_base_link. -->
+  <joint name="apriltag_base_mount_joint" type="fixed">
+    <origin xyz="0.10 0.0 0.05" rpy="0 0 0" />
+    <parent link="volcaniarm_base_link" />
+    <child link="apriltag_base_mount_link" />
+  </joint>
+  <gazebo reference="apriltag_base_mount_joint">
+    <preserveFixedJoint>true</preserveFixedJoint>
+  </gazebo>
+  <joint name="apriltag_base_joint" type="fixed">
+    <origin xyz="0 0 0" rpy="0 ${pi/2} 0" />
+    <parent link="apriltag_base_mount_link" />
+    <child link="apriltag_base_link" />
+  </joint>
+  <gazebo reference="apriltag_base_joint">
     <preserveFixedJoint>true</preserveFixedJoint>
   </gazebo>

Commit message: Polish: world fixed frame, base tag past table, always-home cycle
RViz config (calibration_dashboard.rviz)
- Fixed Frame is now world (was volcaniarm_base_link).
- Drop the Selection / Tool Properties / Views panels and hide the
  right dock for a cleaner left-only layout.

URDF (volcaniarm_apriltag.xacro)
- Bump the base AprilTag mount along volcaniarm_base_link +X from
  0.10 to 0.65 so the tag clears the table footprint and is visible
  to the camera. Y/Z relative to base_link unchanged. Comment notes
  the offset is still pending physical measurement.

Runner (calibration_runner.py)
- The arm now always homes before the first visit and after every
  visit, regardless of test type. Each iteration is one full
  home -> preview -> approve -> target -> measure -> home cycle, so
  multi-iteration single-target runs interleave returns to home as
  intended. The legacy return_home_between_targets flag is no longer
  the gating predicate.

Dashboard widget (calibration_dashboard_widget.py)
- New home theta_right / home theta_left spinboxes (radians, range
  [-pi, pi], default 0.0). Their values populate
  RunRequest.home_position so the home pose can be tuned per run.
  Saved/restored via plugin_settings like the rest of the form.

File: src/volcaniarm_description/urdf/volcaniarm_apriltag.xacro (robot description, xacro)
@@ -76,8 +76,11 @@
     </inertial>
   </link>
-  <!-- TODO(thesis): replace with the measured mount offset once the
-       printed bracket is fitted on volcaniarm_base_link. -->
+  <!-- Pushed out along volcaniarm_base_link +X so the tag clears the
+       table footprint and stays visible to the camera. Y/Z relative
+       to base_link are unchanged.
+       TODO(thesis): replace with the measured mount offset once the
+       printed bracket is fitted. -->
   <joint name="apriltag_base_mount_joint" type="fixed">
-    <origin xyz="0.10 0.0 0.05" rpy="0 0 0" />
+    <origin xyz="0.65 0.0 0.05" rpy="0 0 0" />
     <parent link="volcaniarm_base_link" />
     <child link="apriltag_base_mount_link" />

Commit message: Reposition + widen calibration camera, extend EE tag mount
sim_bringup now auto-defaults world_name to 'calibration' (lab world
minus the potted plant) when calibration:=true, still overridable.

The calibration camera moves from base_link xyz=(2.0, 0, -0.48) to
xyz=(1.5, 0, -0.08) so its world Z sits at the workspace midpoint and
the standoff is short enough that the table base fills more of the
frame. Sim camera intrinsics widen from 1.25 rad / 848x480 to 1.5 rad
/ 1280x720 so the full home-to-high-target envelope fits in a single
frame with the EE apriltag still ~55 px wide at 1.5 m. Comments note
this diverges from the real D435 spec.

EE apriltag mount xyz extends from 0.04 to 0.1 along right_arm_tip_link
+X, which at home points back along the camera optical axis, so the
tag sits closer to the camera without shifting in image Y/Z (calibration
residuals unchanged).

File: src/volcaniarm_description/urdf/volcaniarm_apriltag.xacro (robot description, xacro)
@@ -33,6 +33,13 @@
     </inertial>
   </link>
+  <!-- Mount offset in right_arm_tip_link frame. The tip's +X axis at
+       home points back along the calibration-camera optical axis (i.e.
+       perpendicular to the arm's working Y-Z plane), so extending the
+       offset along +X brings the tag closer to the camera *without*
+       moving it in image Y/Z and without affecting the calibration's
+       Y-Z residuals. The mount roll keeps the printed bracket aimed
+       roughly upward at the camera at typical operating poses. -->
   <joint name="apriltag_ee_mount_joint" type="fixed">
-    <origin xyz="0.04 0 0" rpy="${-pi/3.4} 0 0" />
+    <origin xyz="0.1 0 0" rpy="${-pi/3.4} 0 0" />
     <parent link="right_arm_tip_link" />
     <child link="apriltag_ee_mount_link" />

File: src/volcaniarm_description/urdf/volcaniarm_gazebo.xacro (robot description, xacro)
@@ -7,12 +7,22 @@
     </plugin>
   </gazebo>
-  <!-- RGBD Camera sensor -->
+  <!-- RGBD Camera sensor.
+       HFOV 1.5 rad (~86 deg) and 1280x720 resolution intentionally
+       diverge from the real D435 color spec (~69 deg HFOV at 848x480)
+       to widen the calibration camera's coverage so the full EE
+       operating envelope (home tip near world Z=0.23 to high targets
+       near Z=1.58) fits in a single frame at 2.5 m standoff. The
+       higher resolution keeps the 0.2 m sim apriltags at ~55 px wide
+       at 2.5 m (down to ~6 px per bit, comfortably above the 36h11
+       decode floor). For a sim-vs-real apples-to-apples comparison
+       on a calibrated D435, drop these back to 1.25 / 848x480 and
+       reposition the camera. -->
   <gazebo reference="camera_link">
       <sensor name="rgbd_camera" type="rgbd_camera">
           <camera>
-              <horizontal_fov>1.25</horizontal_fov>
+              <horizontal_fov>1.5</horizontal_fov>
               <image>
-                  <width>848</width>
-                  <height>480</height>
+                  <width>1280</width>
+                  <height>720</height>
               </image>
               <clip>

File: src/volcaniarm_description/urdf/volcaniarm_realsense.xacro (robot description, xacro)
@@ -3,15 +3,19 @@
   <!-- Calibration mode: horizontal camera in front of the robot (sim only).
        base_link is at world (0,0,0.98) with yaw=pi, so base_link +X is
-       world -X. xyz=(2.0, 0, -0.48) -> world (-2.0, 0, 0.5); yaw=pi
-       points +X back toward world +X. Z is set near the midpoint of the
-       EE-tag and base-tag world heights so both fit in the vertical FOV.
-       NOTE: at home (theta=0,0) the EE tag normal points world +Z, so a
-       horizontal camera sees that tag edge-on and apriltag will not
-       decode it. Detection of the EE tag becomes reliable as soon as
-       the arm starts moving. If you need home-pose EE detection, tilt
-       the camera downward or rotate the EE tag mount. -->
+       world -X. xyz=(2.5, 0, -0.07) -> world (-2.5, 0, 0.91); yaw=pi
+       points +X back toward world +X.
+       Camera Z (0.91 m) is the midpoint of the workspace vertical
+       range (home tip near world Z=0.23, high targets near Z=1.58),
+       and the X distance (2.5 m) is set so the sim camera vertical
+       FOV of ~45 deg covers the full 1.55 m workspace span (with
+       0.2 m tag size accounted for) and keeps the entire EE tag
+       inside the image at every test pose. At 2 m distance the FOV
+       was ~0.24 m short and high-target captures lost the EE tag
+       to the top of the frame; pulling the camera back trades a
+       smaller tag in the image (~48 px wide vs ~62) for full
+       coverage of the operating envelope. -->
   <xacro:if value="$(arg calibration)">
     <joint name="calibration_camera_joint" type="fixed">
-      <origin xyz="2.0 0 -0.48" rpy="0 0 ${pi}" />
+      <origin xyz="1.8 0 -0.06" rpy="0 0 ${pi}" />
       <parent link="base_link" />
       <child link="camera_link" />

Commit message: Tune AprilTag mount offsets to match the printed brackets
EE tag: pull the X offset on right_arm_tip_link in from 0.1 to 0.02 m.
Base tag: drop the Z offset on volcaniarm_base_link from +0.05 to -0.03 m.

File: src/volcaniarm_description/urdf/volcaniarm_apriltag.xacro (robot description, xacro)
@@ -45,5 +45,5 @@
        roughly upward at the camera at typical operating poses. -->
   <joint name="apriltag_ee_mount_joint" type="fixed">
-    <origin xyz="0.1 0 0" rpy="${-pi/3.4} 0 0" />
+    <origin xyz="0.02 0 0" rpy="${-pi/3.4} 0 0" />
     <parent link="right_arm_tip_link" />
     <child link="apriltag_ee_mount_link" />
@@ -93,5 +93,5 @@
        printed bracket is fitted. -->
   <joint name="apriltag_base_mount_joint" type="fixed">
-    <origin xyz="0.65 0.0 0.05" rpy="0 0 0" />
+    <origin xyz="0.65 0.0 -0.03" rpy="0 0 0" />
     <parent link="volcaniarm_base_link" />
     <child link="apriltag_base_mount_link" />

Commit message: Edit urdf apriltag marker pose

File: src/volcaniarm_description/urdf/volcaniarm_apriltag.xacro (robot description, xacro)
@@ -55,5 +55,5 @@
     <!-- Tag face pointing in +X. The DAE quad face is on the Z plane,
          so rotate 90 deg around Y to face +X. -->
-    <origin xyz="0 0 0" rpy="0 ${pi/2} 0" />
+    <origin xyz="0.02 0 0" rpy="0 ${pi/2} 0" />
     <parent link="apriltag_ee_mount_link" />
     <child link="apriltag_ee_link" />
