Commit message: Add end effector controller node

File: src/volcaniarm_description/urdf/volcaniarm.urdf.xacro (robot description, xacro)
@@ -9,5 +9,5 @@
   <link name="world" />
   <joint name="world_to_base" type="fixed">
-    <origin xyz="0 0 1" rpy="0 0 0" />
+    <origin xyz="0 0 1.2" rpy="0 0 0" />
     <parent link="world" />
     <child link="delta_arm_base_link" />

Commit message: Edit volcaniarm_end_effector_marker.py. Now showing the marker path correctly

File: src/volcaniarm_description/urdf/volcaniarm.urdf.xacro (robot description, xacro)
@@ -9,5 +9,5 @@
   <link name="world" />
   <joint name="world_to_base" type="fixed">
-    <origin xyz="0 0 1.2" rpy="0 0 0" />
+    <origin xyz="0 0 1.3" rpy="0 0 0" />
     <parent link="world" />
     <child link="delta_arm_base_link" />

Commit message: Edit urdf with new coordinate system

File: src/volcaniarm_description/urdf/volcaniarm.urdf.xacro (robot description, xacro)
@@ -9,5 +9,5 @@
   <link name="world" />
   <joint name="world_to_base" type="fixed">
-    <origin xyz="0 0 1.3" rpy="0 0 0" />
+    <origin xyz="0 0 1.3" rpy="3.14 0 0" />
     <parent link="world" />
     <child link="delta_arm_base_link" />
@@ -18,15 +18,15 @@
     <inertial>
       <origin
-        xyz="0.044852 5.6163E-11 -0.047504"
-        rpy="0 0 0" />
-      <mass
-        value="3.6689" />
-      <inertia
-        ixx="0.037076"
-        ixy="-5.2217E-06"
-        ixz="-0.00045503"
-        iyy="0.0099763"
-        iyz="-2.5372E-12"
-        izz="0.042777" />
+        xyz="0.0448523615659837 -5.61618529459906E-11 0.0475041838279733"
+        rpy="0 0 0" />
+      <mass
+        value="3.66893125370708" />
+      <inertia
+        ixx="0.0370764826444317"
+        ixy="5.22170430710044E-06"
+        ixz="0.000455029302088239"
+        iyy="0.00997633418242008"
+        iyz="-2.53723287794529E-12"
+        izz="0.042776927188676" />
     </inertial>
     <visual>
@@ -59,15 +59,15 @@
     <inertial>
       <origin
-        xyz="0.034442 0.0032708 -0.20791"
-        rpy="0 0 0" />
-      <mass
-        value="0.25563" />
-      <inertia
-        ixx="0.0015999"
-        ixy="-2.5707E-06"
-        ixz="4.8958E-07"
-        iyy="0.0016014"
-        iyz="2.7775E-06"
-        izz="8.8967E-05" />
+        xyz="0.0344418579623738 0.207911851059774 0.00327083348162716"
+        rpy="0 0 0" />
+      <mass
+        value="0.255626035233683" />
+      <inertia
+        ixx="0.00159990350392906"
+        ixy="-4.89579235407502E-07"
+        ixz="-2.57067549462293E-06"
+        iyy="8.89672102610009E-05"
+        iyz="-2.77751340707856E-06"
+        izz="0.00160137777854202" />
     </inertial>
     <visual>
@@ -99,5 +99,5 @@
     type="revolute">
     <origin
-      xyz="0.1825 -0.215 -0.0582"
+      xyz="0.1825 0.215 0.0582"
       rpy="0 0 0" />
     <parent
@@ -118,15 +118,15 @@
     <inertial>
       <origin
-        xyz="0.034442 -0.00032898 -0.20791"
-        rpy="0 0 0" />
-      <mass
-        value="0.25563" />
-      <inertia
-        ixx="0.0015999"
-        ixy="-2.5707E-06"
-        ixz="4.8958E-07"
-        iyy="0.0016014"
-        iyz="-4.1043E-06"
-        izz="8.8968E-05" />
+        xyz="0.0344418579623738 0.207911854085233 -0.000328981745472023"
+        rpy="0 0 0" />
+      <mass
+        value="0.255626035233677" />
+      <inertia
+        ixx="0.00159990350392901"
+        ixy="-4.89578784056069E-07"
+        ixz="-2.57068360841827E-06"
+        iyy="8.89679482853774E-05"
+        iyz="4.10433625636923E-06"
+        izz="0.00160137704051758" />
     </inertial>
     <visual>
@@ -158,5 +158,5 @@
     type="revolute">
     <origin
-      xyz="0.1825 0.215 -0.0582"
+      xyz="0.1825 -0.215 0.0582"
       rpy="0 0 0" />
     <parent
@@ -207,21 +207,20 @@
     <child link="camera_link_optical" />
   </joint>
-  <!-- STRAT BREAK -->
-<!--
-  <link
+  <!-- right arm -->
+  <!-- <link
     name="right_arm_link">
     <inertial>
       <origin
-        xyz="-2.2204E-16 -0.019365 -0.31121"
-        rpy="0 0 0" />
-      <mass
-        value="0.31139" />
-      <inertia
-        ixx="0.0060642"
-        ixy="-1.1232E-13"
-        ixz="7.512E-14"
-        iyy="0.0060587"
-        iyz="1.0603E-13"
-        izz="0.00011844" />
+        xyz="-6.66133814775094E-16 0.311213203465175 -0.0193654158244768"
+        rpy="0 0 0" />
+      <mass
+        value="0.311388968904969" />
+      <inertia
+        ixx="0.00606416863421189"
+        ixy="-7.51196529191669E-14"
+        ixz="-1.12323620344002E-13"
+        iyy="0.000118443044081191"
+        iyz="-1.06032881991769E-13"
+        izz="0.00605866068599566" />
     </inertial>
     <visual>
@@ -236,5 +235,5 @@
         name="">
         <color
-          rgba="0.79216 0.81961 0.93333 1" />
+          rgba="0.792156862745098 0.819607843137255 0.933333333333333 1" />
       </material>
     </visual>
@@ -253,5 +252,5 @@
     type="revolute">
     <origin
-      xyz="0.042 0.02 -0.41621"
+      xyz="0.042 0.41621 0.02"
       rpy="0.31866 0 0" />
     <parent
@@ -266,20 +265,21 @@
       effort="10"
       velocity="10" />
-  </joint>
-  <link
+  </joint> -->
+  <!-- left arm -->
+  <!-- <link
     name="left_arm_link">
     <inertial>
       <origin
-        xyz="0.00010961 0.018304 -0.32828"
-        rpy="0 0 0" />
-      <mass
-        value="0.32945" />
-      <inertia
-        ixx="0.0060651"
-        ixy="4.5433E-12"
-        ixz="-3.103E-12"
-        iyy="0.0060639"
-        iyz="-3.0489E-09"
-        izz="0.00012364" />
+        xyz="0.000109605665534085 0.328277798613676 0.0183035870311327"
+        rpy="0 0 0" />
+      <mass
+        value="0.329453720362959" />
+      <inertia
+        ixx="0.00606509659166047"
+        ixy="3.1029743207609E-12"
+        ixz="4.54332710534137E-12"
+        iyy="0.000123636511114911"
+        iyz="3.04888853494377E-09"
+        izz="0.00606385685806373" />
     </inertial>
     <visual>
@@ -294,5 +294,5 @@
         name="">
         <color
-          rgba="0.79216 0.81961 0.93333 1" />
+          rgba="0.792156862745098 0.819607843137255 0.933333333333333 1" />
       </material>
     </visual>
@@ -311,5 +311,5 @@
     type="revolute">
     <origin
-      xyz="0.042 -0.02 -0.41621"
+      xyz="0.042 0.41621 -0.02"
       rpy="-0.31866 0 0" />
     <parent
@@ -325,4 +325,3 @@
       velocity="10" />
   </joint> -->
-  <!-- END BREAK -->
 </robot>

Commit message: Fix FK

File: src/volcaniarm_description/urdf/volcaniarm.urdf.xacro (robot description, xacro)
@@ -9,5 +9,5 @@
   <link name="world" />
   <joint name="world_to_base" type="fixed">
-    <origin xyz="0 0 1.3" rpy="3.14 0 0" />
+    <origin xyz="0 0 1.3" rpy="3.14159 0 0" />
     <parent link="world" />
     <child link="delta_arm_base_link" />

File: src/volcaniarm_description/urdf/volcaniarm_ros2_control.xacro (robot description, xacro)
@@ -9,4 +9,5 @@
         <!-- ros2_control Common Interfaces -->
         <joint name="right_elbow_joint">
+            <param name="initial_position">1.57</param>
             <command_interface name="position">
               <param name="min">-2.09</param>
@@ -17,4 +18,5 @@
         </joint>
         <joint name="left_elbow_joint">
+            <param name="initial_position">1.57</param>
             <command_interface name="position">
               <param name="min">-2.09</param>

Commit message: Fix depth camera position

File: src/volcaniarm_description/urdf/volcaniarm.urdf.xacro (robot description, xacro)
@@ -9,5 +9,5 @@
   <link name="world" />
   <joint name="world_to_base" type="fixed">
-    <origin xyz="0 0 1.3" rpy="3.14159 0 0" />
+    <origin xyz="0 0 1.0" rpy="3.14159 0 0" />
     <parent link="world" />
     <child link="delta_arm_base_link" />
@@ -196,5 +196,5 @@
   </link>
   <joint name="camera_joint" type="fixed">
-    <origin xyz="0.5 0 0.1" rpy="0 1.7 0" />
+    <origin xyz="0.5 0 0.1" rpy="0 -1.8 0" />
     <parent link="delta_arm_base_link" />
     <child link="camera_link" />
