Commit message: Add closed loop kinematics to the model. Camera & passive joints frames still need to be fixed

File: src/volcaniarm_description/urdf/volcaniarm.urdf.xacro (robot description, xacro)
@@ -11,193 +11,627 @@
   <link name="world" />
   <joint name="world_to_base" type="fixed">
-    <origin xyz="0 0 1.0" rpy="3.14159 0 0" />
+    <origin xyz="0 0 0.98" rpy="0 0 3.14159" />
     <parent link="world" />
-    <child link="delta_arm_base_link" />
-  </joint>
-  <!-- base -->
-  <link
-    name="delta_arm_base_link">
-    <inertial>
-      <origin
-        xyz="0.0448523615659837 -5.61618529459906E-11 0.0475041838279733"
-        rpy="0 0 0" />
-      <mass
-        value="3.66893125370708" />
-      <inertia
-        ixx="0.0370764826444317"
-        ixy="5.22170430710044E-06"
-        ixz="0.000455029302088239"
-        iyy="0.00997633418242008"
-        iyz="-2.53723287794529E-12"
-        izz="0.042776927188676" />
-    </inertial>
-    <visual>
-      <origin
-        xyz="0 0 0"
-        rpy="0 0 0" />
-      <geometry>
-        <mesh
-          filename="package://volcaniarm_description/meshes/delta_arm_base_link.STL" />
-      </geometry>
-      <material
-        name="">
-        <color
-          rgba="0.79216 0.81961 0.93333 1" />
-      </material>
-    </visual>
-    <collision>
-      <origin
-        xyz="0 0 0"
-        rpy="0 0 0" />
-      <geometry>
-        <mesh
-          filename="package://volcaniarm_description/meshes/delta_arm_base_link.STL" />
-      </geometry>
-    </collision>
-  </link>
-  <!-- right elbow -->
-  <link
-    name="right_elbow_link">
-    <inertial>
-      <origin
-        xyz="0.0344418579623738 0.207911851059774 0.00327083348162716"
-        rpy="0 0 0" />
-      <mass
-        value="0.255626035233683" />
-      <inertia
-        ixx="0.00159990350392906"
-        ixy="-4.89579235407502E-07"
-        ixz="-2.57067549462293E-06"
-        iyy="8.89672102610009E-05"
-        iyz="-2.77751340707856E-06"
-        izz="0.00160137777854202" />
-    </inertial>
-    <visual>
-      <origin
-        xyz="0 0 0"
-        rpy="0 0 0" />
-      <geometry>
-        <mesh
-          filename="package://volcaniarm_description/meshes/right_elbow_link.STL" />
-      </geometry>
-      <material
-        name="">
-        <color
-          rgba="0.79216 0.81961 0.93333 1" />
-      </material>
-    </visual>
-    <collision>
-      <origin
-        xyz="0 0 0"
-        rpy="0 0 0" />
-      <geometry>
-        <mesh
-          filename="package://volcaniarm_description/meshes/right_elbow_link.STL" />
-      </geometry>
-    </collision>
-  </link>
-  <joint
-    name="right_elbow_joint"
-    type="revolute">
-    <origin
-      xyz="0.1825 0.215 0.0582"
-      rpy="0 0 0" />
-    <parent
-      link="delta_arm_base_link" />
-    <child
-      link="right_elbow_link" />
-    <axis
-      xyz="1 0 0" />
-    <limit
-      lower="-3.14"
-      upper="3.14"
-      effort="10"
-      velocity="10" />
-  </joint>
-  <!-- left elbow -->
-  <link
-    name="left_elbow_link">
-    <inertial>
-      <origin
-        xyz="0.0344418579623738 0.207911854085233 -0.000328981745472023"
-        rpy="0 0 0" />
-      <mass
-        value="0.255626035233677" />
-      <inertia
-        ixx="0.00159990350392901"
-        ixy="-4.89578784056069E-07"
-        ixz="-2.57068360841827E-06"
-        iyy="8.89679482853774E-05"
-        iyz="4.10433625636923E-06"
-        izz="0.00160137704051758" />
-    </inertial>
-    <visual>
-      <origin
-        xyz="0 0 0"
-        rpy="0 0 0" />
-      <geometry>
-        <mesh
-          filename="package://volcaniarm_description/meshes/left_elbow_link.STL" />
-      </geometry>
-      <material
-        name="">
-        <color
-          rgba="0.79216 0.81961 0.93333 1" />
-      </material>
-    </visual>
-    <collision>
-      <origin
-        xyz="0 0 0"
-        rpy="0 0 0" />
-      <geometry>
-        <mesh
-          filename="package://volcaniarm_description/meshes/left_elbow_link.STL" />
-      </geometry>
-    </collision>
-  </link>
-  <joint
-    name="left_elbow_joint"
-    type="revolute">
-    <origin
-      xyz="0.1825 -0.215 0.0582"
-      rpy="0 0 0" />
-    <parent
-      link="delta_arm_base_link" />
-    <child
-      link="left_elbow_link" />
-    <axis
-      xyz="1 0 0" />
-    <limit
-      lower="-3.14"
-      upper="3.14"
-      effort="10"
-      velocity="10" />
-  </joint>
-  <!-- Camera link -->
+    <child link="base_link" />
+  </joint>
+  <!-- base (table top) -->
+  <link name="base_link">
+    <inertial>
+      <origin xyz="0.0033183 1.7612E-06 -0.24794" rpy="0 0 0" />
+      <mass value="5.4796" />
+      <inertia ixx="0.36605" ixy="-2.0049E-09" ixz="1.5542E-08"
+               iyy="0.19294" iyz="-3.1213E-09" izz="0.31414" />
+    </inertial>
+    <visual>
+      <origin xyz="0 0 0" rpy="0 0 0" />
+      <geometry>
+        <mesh filename="package://volcaniarm_description/meshes/base_link.STL" />
+      </geometry>
+      <material name="">
+        <color rgba="1 0 0 1" />
+      </material>
+    </visual>
+    <collision>
+      <origin xyz="0 0 0" rpy="0 0 0" />
+      <geometry>
+        <mesh filename="package://volcaniarm_description/meshes/base_link.STL" />
+      </geometry>
+    </collision>
+  </link>
+  <!-- ======================== TABLE LEGS ======================== -->
+  <!-- Front-left table leg -->
+  <link name="fl_table_leg_link">
+    <inertial>
+      <origin xyz="0 2.2204E-16 0.22347" rpy="0 0 0" />
+      <mass value="0.15157" />
+      <inertia ixx="0.0028107" ixy="-1.2462E-19" ixz="-4.3818E-20"
+               iyy="0.0028135" iyz="-1.2312E-20" izz="5.0184E-05" />
+    </inertial>
+    <visual>
+      <origin xyz="0 0 0" rpy="0 0 0" />
+      <geometry>
+        <mesh filename="package://volcaniarm_description/meshes/fl_table_leg_link.STL" />
+      </geometry>
+      <material name="">
+        <color rgba="0.79216 0.81961 0.93333 1" />
+      </material>
+    </visual>
+    <collision>
+      <origin xyz="0 0 0" rpy="0 0 0" />
+      <geometry>
+        <mesh filename="package://volcaniarm_description/meshes/fl_table_leg_link.STL" />
+      </geometry>
+    </collision>
+  </link>
+  <joint name="fl_table_leg_joint" type="fixed">
+    <origin xyz="0.340000000000002 0.697999999999994 -0.883" rpy="0 0 0" />
+    <parent link="base_link" />
+    <child link="fl_table_leg_link" />
+  </joint>
+  <!-- FL caster wheel mount -->
+  <link name="fl_caster_wheel_mount_link">
+    <inertial>
+      <origin xyz="-0.011459 -7.0567E-09 -0.011665" rpy="0 0 0" />
+      <mass value="0.047319" />
+      <inertia ixx="1.6675E-05" ixy="-8.0944E-11" ixz="-8.1003E-07"
+               iyy="2.9049E-05" iyz="-7.8988E-11" izz="3.76E-05" />
+    </inertial>
+    <visual>
+      <origin xyz="0 0 0" rpy="0 0 0" />
+      <geometry>
+        <mesh filename="package://volcaniarm_description/meshes/fl_caster_wheel_mount_link.STL" />
+      </geometry>
+      <material name="">
+        <color rgba="0.79216 0.81961 0.93333 1" />
+      </material>
+    </visual>
+    <collision>
+      <origin xyz="0 0 0" rpy="0 0 0" />
+      <geometry>
+        <mesh filename="package://volcaniarm_description/meshes/fl_caster_wheel_mount_link.STL" />
+      </geometry>
+    </collision>
+  </link>
+  <joint name="fl_caster_wheel_mount_joint" type="fixed">
+    <origin xyz="0 0 0" rpy="0 0 0" />
+    <parent link="fl_table_leg_link" />
+    <child link="fl_caster_wheel_mount_link" />
+  </joint>
+  <!-- FL caster wheel -->
+  <link name="fl_caster_wheel_link">
+    <inertial>
+      <origin xyz="0 -5.3545E-05 -1.1102E-16" rpy="0 0 0" />
+      <mass value="0.12084" />
+      <inertia ixx="4.6943E-05" ixy="2.8182E-17" ixz="-1.6458E-15"
+               iyy="7.6353E-05" iyz="4.9423E-17" izz="4.6943E-05" />
+    </inertial>
+    <visual>
+      <origin xyz="0 0 0" rpy="0 0 0" />
+      <geometry>
+        <mesh filename="package://volcaniarm_description/meshes/fl_caster_wheel_link.STL" />
+      </geometry>
+      <material name="">
+        <color rgba="0.79216 0.81961 0.93333 1" />
+      </material>
+    </visual>
+    <collision>
+      <origin xyz="0 0 0" rpy="0 0 0" />
+      <geometry>
+        <mesh filename="package://volcaniarm_description/meshes/fl_caster_wheel_link.STL" />
+      </geometry>
+    </collision>
+  </link>
+  <joint name="fl_caster_wheel_joint" type="fixed">
+    <origin xyz="-0.0324999999999998 0 -0.0595000000000001" rpy="0 0 0" />
+    <parent link="fl_caster_wheel_mount_link" />
+    <child link="fl_caster_wheel_link" />
+  </joint>
+  <!-- Front-right table leg -->
+  <link name="fr_table_leg_link">
+    <inertial>
+      <origin xyz="-4.4409E-16 -5.5511E-17 0.22347" rpy="0 0 0" />
+      <mass value="0.15157" />
+      <inertia ixx="0.0028107" ixy="-2.7017E-19" ixz="2.3161E-21"
+               iyy="0.0028135" iyz="-2.0835E-19" izz="5.0184E-05" />
+    </inertial>
+    <visual>
+      <origin xyz="0 0 0" rpy="0 0 0" />
+      <geometry>
+        <mesh filename="package://volcaniarm_description/meshes/fr_table_leg_link.STL" />
+      </geometry>
+      <material name="">
+        <color rgba="0.79216 0.81961 0.93333 1" />
+      </material>
+    </visual>
+    <collision>
+      <origin xyz="0 0 0" rpy="0 0 0" />
+      <geometry>
+        <mesh filename="package://volcaniarm_description/meshes/fr_table_leg_link.STL" />
+      </geometry>
+    </collision>
+  </link>
+  <joint name="fr_table_leg_joint" type="fixed">
+    <origin xyz="0.340000000000005 -0.697999999999998 -0.883" rpy="0 0 0" />
+    <parent link="base_link" />
+    <child link="fr_table_leg_link" />
+  </joint>
+  <!-- FR caster wheel mount -->
+  <link name="fr_caster_wheel_mount_link">
+    <inertial>
+      <origin xyz="-0.011459 -7.0567E-09 -0.011665" rpy="0 0 0" />
+      <mass value="0.047319" />
+      <inertia ixx="1.6675E-05" ixy="-8.0944E-11" ixz="-8.1003E-07"
+               iyy="2.9049E-05" iyz="-7.8988E-11" izz="3.76E-05" />
+    </inertial>
+    <visual>
+      <origin xyz="0 0 0" rpy="0 0 0" />
+      <geometry>
+        <mesh filename="package://volcaniarm_description/meshes/fr_caster_wheel_mount_link.STL" />
+      </geometry>
+      <material name="">
+        <color rgba="0.79216 0.81961 0.93333 1" />
+      </material>
+    </visual>
+    <collision>
+      <origin xyz="0 0 0" rpy="0 0 0" />
+      <geometry>
+        <mesh filename="package://volcaniarm_description/meshes/fr_caster_wheel_mount_link.STL" />
+      </geometry>
+    </collision>
+  </link>
+  <joint name="fr_caster_wheel_mount_joint" type="fixed">
+    <origin xyz="0 0 0" rpy="0 0 0" />
+    <parent link="fr_table_leg_link" />
+    <child link="fr_caster_wheel_mount_link" />
+  </joint>
+  <!-- FR caster wheel -->
+  <link name="fr_caster_wheel_link">
+    <inertial>
+      <origin xyz="0 -5.3545E-05 0" rpy="0 0 0" />
+      <mass value="0.12084" />
+      <inertia ixx="4.6943E-05" ixy="2.8345E-17" ixz="-1.6458E-15"
+               iyy="7.6353E-05" iyz="4.9116E-17" izz="4.6943E-05" />
+    </inertial>
+    <visual>
+      <origin xyz="0 0 0" rpy="0 0 0" />
+      <geometry>
+        <mesh filename="package://volcaniarm_description/meshes/fr_caster_wheel_link.STL" />
+      </geometry>
+      <material name="">
+        <color rgba="0.79216 0.81961 0.93333 1" />
+      </material>
+    </visual>
+    <collision>
+      <origin xyz="0 0 0" rpy="0 0 0" />
+      <geometry>
+        <mesh filename="package://volcaniarm_description/meshes/fr_caster_wheel_link.STL" />
+      </geometry>
+    </collision>
+  </link>
+  <joint name="fr_caster_wheel_joint" type="fixed">
+    <origin xyz="-0.0324999999999998 0 -0.0594999999999999" rpy="0 0 0" />
+    <parent link="fr_caster_wheel_mount_link" />
+    <child link="fr_caster_wheel_link" />
+  </joint>
+  <!-- Rear-left table leg -->
+  <link name="rl_table_leg_link">
+    <inertial>
+      <origin xyz="2.2204E-16 4.4409E-16 0.22347" rpy="0 0 0" />
+      <mass value="0.15157" />
+      <inertia ixx="0.0028107" ixy="-6.6369E-21" ixz="3.4765E-19"
+               iyy="0.0028135" iyz="-1.384E-18" izz="5.0184E-05" />
+    </inertial>
+    <visual>
+      <origin xyz="0 0 0" rpy="0 0 0" />
+      <geometry>
+        <mesh filename="package://volcaniarm_description/meshes/rl_table_leg_link.STL" />
+      </geometry>
+      <material name="">
+        <color rgba="0.79216 0.81961 0.93333 1" />
+      </material>
+    </visual>
+    <collision>
+      <origin xyz="0 0 0" rpy="0 0 0" />
+      <geometry>
+        <mesh filename="package://volcaniarm_description/meshes/rl_table_leg_link.STL" />
+      </geometry>
+    </collision>
+  </link>
+  <joint name="rl_table_leg_joint" type="fixed">
+    <origin xyz="-0.340000000000005 0.697999999999997 -0.883" rpy="0 0 0" />
+    <parent link="base_link" />
+    <child link="rl_table_leg_link" />
+  </joint>
+  <!-- RL caster wheel mount -->
+  <link name="rl_caster_wheel_mount_link">
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
File: src/volcaniarm_description/urdf/volcaniarm_gazebo.xacro (robot description, xacro)
@@ -7,23 +7,38 @@
     </plugin>
   </gazebo>
-    <gazebo reference="camera_link">
-        <sensor name="rgbd_camera" type="rgbd_camera">
-            <camera>
-                <horizontal_fov>1.25</horizontal_fov>
-                <image>
-                    <width>848</width>
-                    <height>480</height>
-                </image>
-                <clip>
-                    <near>0.3</near>
-                    <far>15</far>
-                </clip>
-            </camera>
-            <always_on>1</always_on>
-            <update_rate>30</update_rate>
-            <visualize>true</visualize>
-            <topic>rgbd_camera</topic>
-            <gz_frame_id>camera_link</gz_frame_id>
-        </sensor>
-    </gazebo>
+  <!-- RGBD Camera sensor -->
+  <gazebo reference="camera_link">
+      <sensor name="rgbd_camera" type="rgbd_camera">
+          <camera>
+              <horizontal_fov>1.25</horizontal_fov>
+              <image>
+                  <width>848</width>
+                  <height>480</height>
+              </image>
+              <clip>
+                  <near>0.3</near>
+                  <far>15</far>
+              </clip>
+          </camera>
+          <always_on>1</always_on>
+          <update_rate>30</update_rate>
+          <visualize>true</visualize>
+          <topic>rgbd_camera</topic>
+          <gz_frame_id>camera_link</gz_frame_id>
+      </sensor>
+  </gazebo>
+  <!-- DetachableJoint: closes the 5-bar loop at runtime -->
+  <gazebo>
+    <plugin filename="libgz-sim-detachable-joint-system.so"
+            name="gz::sim::systems::DetachableJoint">
+      <parent_link>right_arm_tip_link</parent_link>
+      <child_model>volcaniarm</child_model>
+      <child_link>closure_dummy_link</child_link>
+    </plugin>
+  </gazebo>
+  <!-- Joint state publisher: broadcasts all joint positions back to ROS2 -->
+  <gazebo>
+    <plugin filename="libgz-sim-joint-state-publisher-system.so"
+            name="gz::sim::systems::JointStatePublisher"/>
+  </gazebo>
 </robot>

File: src/volcaniarm_description/urdf/volcaniarm_ros2_control.xacro (robot description, xacro)
@@ -17,5 +17,5 @@
         </hardware>
         <!-- ros2_control Common Interfaces -->
-        <joint name="right_elbow_joint">
+        <joint name="volcaniarm_right_elbow_joint">
             <command_interface name="position">
               <param name="min">-3.14</param>
@@ -23,9 +23,9 @@
             </command_interface>
             <state_interface name="position">
-              <param name="initial_value">1.57</param>
+              <param name="initial_value">0.0</param>
             </state_interface>
             <state_interface name="velocity" />
         </joint>
-        <joint name="left_elbow_joint">
+        <joint name="volcaniarm_left_elbow_joint">
             <command_interface name="position">
               <param name="min">-3.14</param>
@@ -33,5 +33,5 @@
             </command_interface>
             <state_interface name="position">
-              <param name="initial_value">1.57</param>
+              <param name="initial_value">0.0</param>
             </state_interface>
             <state_interface name="velocity" />

Commit message: Fix camera oreintation. Image oreintation need to be fixed still

File: src/volcaniarm_description/urdf/volcaniarm.urdf.xacro (robot description, xacro)
@@ -566,11 +566,8 @@
     </collision>
   </link>
-  <joint name="camera_mount_linear_joint" type="prismatic">
+  <joint name="camera_mount_linear_joint" type="fixed">
     <origin xyz="0.405353761834025 0 0.039999999999992" rpy="0 0 0" />
     <parent link="base_link" />
     <child link="camera_mount_linear_link" />
-    <axis xyz="1 0 0" />
-    <limit lower="-0.3" upper="0.3" effort="10" velocity="10" />
-    <dynamics damping="0.1" friction="0.1" />
   </joint>
   <link name="camera_mount_rev_link">
@@ -582,5 +579,5 @@
     </inertial>
     <visual>
-      <origin xyz="0 0 0" rpy="0 0 0" />
+      <origin xyz="0 0 0" rpy="0 1.5708 0" />
       <geometry>
         <mesh filename="package://volcaniarm_description/meshes/camera_mount_rev_link.STL" />
@@ -591,5 +588,5 @@
     </visual>
     <collision>
-      <origin xyz="0 0 0" rpy="0 0 0" />
+      <origin xyz="0 0 0" rpy="0 1.5708 0" />
       <geometry>
         <mesh filename="package://volcaniarm_description/meshes/camera_mount_rev_link.STL" />
@@ -597,12 +594,9 @@
     </collision>
   </link>
-  <joint name="camera_mount_rev_joint" type="revolute">
+  <joint name="camera_mount_rev_joint" type="fixed">
     <origin xyz="0.192000000000008 0 -0.0290000000000052"
-            rpy="3.14159265358979 0.211904134210419 3.14159265358979" />
+            rpy="3.14159265358979 0.75 3.14159265358979" />
     <parent link="camera_mount_linear_link" />
     <child link="camera_mount_rev_link" />
-    <axis xyz="0 1 0" />
-    <limit lower="-3.14" upper="3.14" effort="10" velocity="10" />
-    <dynamics damping="0.1" friction="0.1" />
   </joint>
   <!-- ======================== CAMERA ======================== -->
@@ -615,5 +609,5 @@
     </inertial>
     <visual>
-      <origin xyz="0 0 0" rpy="0 0 0" />
+      <origin xyz="0 0 0" rpy="0 1.5708 0" />
       <geometry>
         <mesh filename="package://volcaniarm_description/meshes/camera_link.STL" />
@@ -624,5 +618,5 @@
     </visual>
     <collision>
-      <origin xyz="0 0 0" rpy="0 0 0" />
+      <origin xyz="0 0 0" rpy="0 1.5708 0" />
       <geometry>
         <mesh filename="package://volcaniarm_description/meshes/camera_link.STL" />
@@ -631,6 +625,5 @@
   </link>
   <joint name="camera_joint" type="fixed">
-    <origin xyz="-2.37779715432929E-05 0 0.0160004150359285"
-            rpy="0 -0.0135473024600912 0" />
+    <origin xyz="0.0160004150359285 0 0" rpy="0 0 0" />
     <parent link="camera_mount_rev_link" />
     <child link="camera_link" />

Commit message: Fix image oreintatin

File: src/volcaniarm_description/urdf/volcaniarm.urdf.xacro (robot description, xacro)
@@ -625,5 +625,5 @@
   </link>
   <joint name="camera_joint" type="fixed">
-    <origin xyz="0.0160004150359285 0 0" rpy="0 0 0" />
+    <origin xyz="0.0160004150359285 0 0" rpy="3.14159 0 0" />
     <parent link="camera_mount_rev_link" />
     <child link="camera_link" />

Commit message: Add lab.world file

File: src/volcaniarm_description/urdf/volcaniarm.urdf.xacro (robot description, xacro)
@@ -2,4 +2,9 @@
 <robot xmlns:xacro="http://www.ros.org/wiki/xacro" name="volcaniarm">
   <xacro:arg name="use_sim" default="true" />
+  <!-- Camera mount position tuning
+       camera_mount_x range: 0.155 to 0.655
+       camera_mount_pitch: rev joint pitch in radians -->
+  <xacro:property name="camera_mount_x" value="0.25" />
+  <xacro:property name="camera_mount_pitch" value="1.3" />
    <!-- ros2_control hardware interfaces -->
   <xacro:include filename="$(find volcaniarm_description)/urdf/volcaniarm_ros2_control.xacro" />
@@ -567,5 +572,5 @@
   </link>
   <joint name="camera_mount_linear_joint" type="fixed">
-    <origin xyz="0.405353761834025 0 0.039999999999992" rpy="0 0 0" />
+    <origin xyz="${camera_mount_x} 0 0.039999999999992" rpy="0 0 0" />
     <parent link="base_link" />
     <child link="camera_mount_linear_link" />
@@ -596,5 +601,5 @@
   <joint name="camera_mount_rev_joint" type="fixed">
     <origin xyz="0.192000000000008 0 -0.0290000000000052"
-            rpy="3.14159265358979 0.9 3.14159265358979" />
+            rpy="3.14159265358979 ${camera_mount_pitch} 3.14159265358979" />
     <parent link="camera_mount_linear_link" />
     <child link="camera_mount_rev_link" />
