Commit message: Add calibration world, configurable camera, and fix accuracy test
- Create calibration.sdf world (lab without plant)
- Make camera_mount_x/pitch configurable via xacro args through launch chain
- Add calibration mode to URDF: skip arm camera mount, place camera at
  fixed position in front of robot (in volcaniarm_realsense.xacro)
- Scale AprilTag to 200mm for reliable detection in simulation
- Set apriltag detector decimate to 1.0 for full-resolution detection
- Flatten targets list in accuracy_test_params.yaml (ROS 2 YAMLcompat)
- Fix accuracy_test_node to exit cleanly after test completes
- Simplify sim_calibration_bringup to only launch sim stack (tests manual)

File: src/volcaniarm_description/urdf/volcaniarm.urdf.xacro (robot description, xacro)
@@ -3,9 +3,11 @@
   <xacro:arg name="use_sim" default="true" />
   <xacro:arg name="calibration" default="false" />
+  <xacro:arg name="camera_mount_x" default="0.25" />
+  <xacro:arg name="camera_mount_pitch" default="1.3" />
   <!-- Camera mount position tuning
        camera_mount_x range: 0.155 to 0.655
        camera_mount_pitch: rev joint pitch in radians -->
-  <xacro:property name="camera_mount_x" value="0.25" />
-  <xacro:property name="camera_mount_pitch" value="1.3" />
+  <xacro:property name="camera_mount_x" value="$(arg camera_mount_x)" />
+  <xacro:property name="camera_mount_pitch" value="$(arg camera_mount_pitch)" />
    <!-- ros2_control hardware interfaces -->
   <xacro:include filename="$(find volcaniarm_description)/urdf/volcaniarm_ros2_control.xacro" />
@@ -554,4 +556,6 @@
   </joint>
   <!-- ======================== CAMERA MOUNT ======================== -->
+  <!-- Skipped in calibration mode (camera is placed directly by realsense xacro) -->
+  <xacro:unless value="$(arg calibration)">
   <link name="camera_mount_linear_link">
     <inertial>
@@ -610,4 +614,5 @@
     <child link="camera_mount_rev_link" />
   </joint>
+  </xacro:unless>
   <!-- ======================== CAMERA ======================== -->
   <link name="camera_link">
@@ -634,9 +639,11 @@
     </collision>
   </link>
-  <joint name="camera_joint" type="fixed">
-    <origin xyz="0.0160004150359285 0 0" rpy="3.14159 0 0" />
-    <parent link="camera_mount_rev_link" />
-    <child link="camera_link" />
-  </joint>
+  <xacro:unless value="$(arg calibration)">
+    <joint name="camera_joint" type="fixed">
+      <origin xyz="0.0160004150359285 0 0" rpy="3.14159 0 0" />
+      <parent link="camera_mount_rev_link" />
+      <child link="camera_link" />
+    </joint>
+  </xacro:unless>
   <!-- Camera optical frame -->
   <link name="camera_link_optical" />

File: src/volcaniarm_description/urdf/volcaniarm_apriltag.xacro (robot description, xacro)
@@ -2,8 +2,9 @@
 <robot xmlns:xacro="http://www.ros.org/wiki/xacro" name="volcaniarm_apriltag">
   <!-- AprilTag 36h11 ID 20 mounted on the end effector (sim only).
-       The tag is a flat 64mm square facing +X direction.
-       Uses a DAE mesh with baked texture so it renders in both Gazebo and RViz. -->
+       Uses a DAE mesh with baked texture so it renders in both Gazebo and RViz.
+       DAE has 64mm geometry, scaled up to 200mm for reliable detection in sim. -->
   <xacro:property name="tag_mesh"
     value="package://volcaniarm_description/models/Apriltag36_11_00020/apriltag_36h11_id20.dae" />
+  <xacro:property name="tag_scale" value="${0.2 / 0.064}" />
   <!-- Tag visual link attached to right_arm_tip_link -->
   <link name="apriltag_link">
@@ -16,5 +17,5 @@
       <origin xyz="0 0 0" rpy="0 0 0" />
       <geometry>
-        <mesh filename="${tag_mesh}" />
+        <mesh filename="${tag_mesh}" scale="${tag_scale} ${tag_scale} ${tag_scale}" />
       </geometry>
     </visual>

File: src/volcaniarm_description/urdf/volcaniarm_realsense.xacro (robot description, xacro)
@@ -1,7 +1,17 @@
 <?xml version="1.0"?>
 <robot xmlns:xacro="http://www.ros.org/wiki/xacro" name="volcaniarm_realsense">
-  <!-- RealSense D435i camera frames (only when using real hardware) -->
+  <!-- Calibration mode: camera at fixed position in front of robot (sim only).
+       base_link is at world (0,0,0.98) with yaw=pi, so base_link +X = world -X.
+       Camera at world (-1.5, 0, 0.5) facing world +X (toward robot):
+         In base_link frame: xyz=(1.5, 0, -0.48), yaw=pi to face base_link -X = world +X. -->
+  <xacro:if value="$(arg calibration)">
+    <joint name="calibration_camera_joint" type="fixed">
+      <origin xyz="0.8 0 -0.68" rpy="0 0 ${pi}" />
+      <parent link="base_link" />
+      <child link="camera_link" />
+    </joint>
+  </xacro:if>
+  <!-- Real hardware: RealSense D435i extra frames (only when not simulating) -->
   <xacro:unless value="$(arg use_sim)">
-    <!-- RealSense base link -->
     <link name="camera_camera_link" />
     <joint name="camera_to_realsense" type="fixed">
@@ -10,5 +20,4 @@
       <child link="camera_camera_link" />
     </joint>
-    <!-- RealSense depth frame -->
     <link name="camera_depth_frame" />
     <joint name="camera_depth_joint" type="fixed">
@@ -17,5 +26,4 @@
       <child link="camera_depth_frame" />
     </joint>
-    <!-- RealSense depth optical frame -->
     <link name="camera_depth_optical_frame" />
     <joint name="camera_depth_optical_joint" type="fixed">
@@ -24,5 +32,4 @@
       <child link="camera_depth_optical_frame" />
     </joint>
-    <!-- RealSense color frame -->
     <link name="camera_color_frame" />
     <joint name="camera_color_joint" type="fixed">
@@ -31,5 +38,4 @@
       <child link="camera_color_frame" />
     </joint>
-    <!-- RealSense color optical frame -->
     <link name="camera_color_optical_frame" />
     <joint name="camera_color_optical_joint" type="fixed">

Commit message: Default tag_size to 0.064 and plumb through bringup, dashboard, URDF
Real prints are now 64 mm. Detector size and URDF mesh scale both
follow a single tag_size launch arg (default 0.064) forwarded by
real_bringup, sim_bringup, and gazebo.launch.py into the calibration
dashboard include and the xacro Command. Pass tag_size:=0.200 to
revert to the larger prints in either backend; the apriltag mesh
scales proportionally so detector and rendered scene stay in sync.

File: src/volcaniarm_description/urdf/volcaniarm.urdf.xacro (robot description, xacro)
@@ -10,4 +10,8 @@
        Only affects the Gazebo plugin <parameters> blocks. -->
   <xacro:arg name="controller" default="traj" />
+  <!-- AprilTag edge length in metres. Drives both the URDF mesh scale
+       (via volcaniarm_apriltag.xacro) and the apriltag detector size
+       parameter when forwarded by the bringup launches. -->
+  <xacro:arg name="tag_size" default="0.064" />
   <!-- Camera mount position tuning
        camera_mount_x range: 0.155 to 0.655

File: src/volcaniarm_description/urdf/volcaniarm_apriltag.xacro (robot description, xacro)
@@ -3,7 +3,11 @@
   <!-- AprilTag 36h11 markers used for hand-eye calibration and accuracy
        tests. Both tags use a DAE mesh with baked texture so they render
-       in Gazebo and RViz. The DAE has 64mm geometry, scaled up to 200mm
-       for reliable detection in sim. -->
-  <xacro:property name="tag_scale" value="${0.2 / 0.064}" />
+       in Gazebo and RViz. The DAE geometry is 64 mm; the actual rendered
+       size follows the `tag_size` xacro arg (default 0.064 m, i.e. no
+       scaling), with the mesh scaled proportionally. Pass
+       tag_size:=0.200 in the launch file when using the larger printed
+       tags. -->
+  <xacro:property name="tag_size" value="$(arg tag_size)" />
+  <xacro:property name="tag_scale" value="${tag_size / 0.064}" />
   <!-- ============================================================= -->
   <!-- ID 20: end-effector marker (right_arm_tip_link)                -->

Commit message: Apply calibrated camera pose via URDF xacro args, drop static publisher
The previous Phase 1.6 used a static_transform_publisher to override
base_link -> camera_link with the calibrated pose. That fights the
URDF's published static for the same edge -- TF2's last-write-wins
made the override unreliable, and gating the URDF's joint to avoid
the conflict orphaned camera_link in the URDF tree (robot disappeared
from RViz).

URDF: camera_joint origin is now parameterised via xacro args
(camera_x/y/z/roll/pitch/yaw, defaults match the original hardcoded
values). Wrapped in a xacro:macro so the same definition applies
in every mode except sim+calibration (where the sim-only
calibration_camera_joint takes over -- now properly gated on
use_sim AND calibration).

real_bringup: reads camera_pose.yaml at launch time and passes
xyz+rpy as xacro args. URDF directly publishes the calibrated edge,
no second publisher, no race. Missing or malformed YAML falls back
to URDF defaults with a warning. The use_camera_pose_config arg is
gone -- delete or rename the YAML to revert.

camera_calibration.py: now computes T(camera_mount_rev_link ->
camera_link) instead of T(base_link -> camera_link), since that's
the URDF edge we parameterise. The override block in the log now
shows xyz+rpy values to paste (or just relaunch). Schema in
camera_pose.yaml reflects the new parent/child frames.

Notebooks: static_accuracy and workspace_coverage now compute
Y-Z-only metrics (Volcaniarm is planar; X is fixed bias) and a
scalar |EE-base| Euclidean distance comparison from FK vs tag --
clean variance, biased absolute, with the bias diagnostic across
goals in workspace_coverage.

File: src/volcaniarm_description/urdf/volcaniarm.urdf.xacro (robot description, xacro)
@@ -5,4 +5,18 @@
   <xacro:arg name="camera_mount_x" default="0.25" />
   <xacro:arg name="camera_mount_pitch" default="1.3" />
+  <!-- camera_joint origin: where camera_link sits relative to
+       camera_mount_rev_link. Defaults match the original URDF's
+       hardcoded values. real_bringup reads config/camera_pose.yaml
+       (written by the calibration dashboard) at launch time and
+       passes the calibrated values as xacro args so the URDF
+       directly reflects the measured camera pose. Active in every
+       mode except sim+calibration, where calibration_camera_joint
+       in volcaniarm_realsense.xacro takes over. -->
+  <xacro:arg name="camera_x" default="0.0160004150359285" />
+  <xacro:arg name="camera_y" default="0.0" />
+  <xacro:arg name="camera_z" default="0.0" />
+  <xacro:arg name="camera_roll" default="3.14159" />
+  <xacro:arg name="camera_pitch" default="0.0" />
+  <xacro:arg name="camera_yaw" default="0.0" />
   <!-- Which controller(s) to load into the Gazebo controller_manager:
        traj = trajectory controller only; policy = RL policy controller only;
@@ -648,11 +662,26 @@
     </collision>
   </link>
-  <xacro:unless value="$(arg calibration)">
+  <!-- camera_joint applies in every mode except sim+calibration, where
+       calibration_camera_joint in volcaniarm_realsense.xacro mounts
+       camera_link directly on base_link to give Gazebo a fixed
+       calibration camera. Origin is parameterised via xacro args so
+       real_bringup can plug in calibrated values from camera_pose.yaml
+       at launch time. -->
+  <xacro:macro name="volcaniarm_camera_joint">
     <joint name="camera_joint" type="fixed">
-      <origin xyz="0.0160004150359285 0 0" rpy="3.14159 0 0" />
+      <origin xyz="$(arg camera_x) $(arg camera_y) $(arg camera_z)"
+              rpy="$(arg camera_roll) $(arg camera_pitch) $(arg camera_yaw)" />
       <parent link="camera_mount_rev_link" />
       <child link="camera_link" />
     </joint>
+  </xacro:macro>
+  <xacro:unless value="$(arg use_sim)">
+    <xacro:volcaniarm_camera_joint />
   </xacro:unless>
+  <xacro:if value="$(arg use_sim)">
+    <xacro:unless value="$(arg calibration)">
+      <xacro:volcaniarm_camera_joint />
+    </xacro:unless>
+  </xacro:if>
   <!-- Camera optical frame -->
   <link name="camera_link_optical" />

File: src/volcaniarm_description/urdf/volcaniarm_realsense.xacro (robot description, xacro)
@@ -15,10 +15,18 @@
        smaller tag in the image (~48 px wide vs ~62) for full
        coverage of the operating envelope. -->
-  <xacro:if value="$(arg calibration)">
-    <joint name="calibration_camera_joint" type="fixed">
-      <origin xyz="1.5 0 -0.5" rpy="0 0 ${pi}" />
-      <parent link="base_link" />
-      <child link="camera_link" />
-    </joint>
+  <!-- Sim-only override for calibration mode: parks the camera 1.5 m
+       in front of the robot facing back so the Gazebo workspace test
+       has a fixed view. On real hardware the camera is mounted on
+       the cart and the URDF's camera_joint (volcaniarm.urdf.xacro)
+       handles the placement, with calibrated values passed via xacro
+       args. -->
+  <xacro:if value="$(arg use_sim)">
+    <xacro:if value="$(arg calibration)">
+      <joint name="calibration_camera_joint" type="fixed">
+        <origin xyz="1.5 0 -0.5" rpy="0 0 ${pi}" />
+        <parent link="base_link" />
+        <child link="camera_link" />
+      </joint>
+    </xacro:if>
   </xacro:if>
   <!-- RealSense D435i frame chain. Published by robot_state_publisher in all

Commit message: Reparent calibration camera to world for off-robot stand setup
In calibration mode the camera is physically removed from the arm and
placed on an external stand, so the URDF can no longer route camera_link
through camera_mount_rev_link. The realsense xacro now emits
calibration_camera_joint with parent=world (sim and real, same logic),
and volcaniarm.urdf.xacro skips the on-robot camera_joint when
calibration is true. Defaults place the stand 1.5 m in front of the arm
(world x=-1.5) at 0.6 m above the floor, looking back toward the robot;
real_bringup forwards the calibrated pose from camera_pose.yaml when
present.

The runner now computes T(world -> camera_link) and persists it under
the matching schema. The RViz config gains a PointCloud2 display so
launching with pointcloud:=true shows the cloud immediately, oriented
correctly via the URDF optical-frame chain.

File: src/volcaniarm_description/urdf/volcaniarm.urdf.xacro (robot description, xacro)
@@ -579,5 +579,8 @@
   </joint>
   <!-- ======================== CAMERA MOUNT ======================== -->
-  <!-- Skipped in calibration mode (camera is placed directly by realsense xacro) -->
+  <!-- Skipped in calibration mode: the camera is physically removed from
+       the robot and placed on an external stand, so calibration_camera_joint
+       in volcaniarm_realsense.xacro parents camera_link directly to
+       base_link instead. -->
   <xacro:unless value="$(arg calibration)">
   <link name="camera_mount_linear_link">
@@ -662,11 +665,12 @@
     </collision>
   </link>
-  <!-- camera_joint applies in every mode except sim+calibration, where
-       calibration_camera_joint in volcaniarm_realsense.xacro mounts
-       camera_link directly on base_link to give Gazebo a fixed
-       calibration camera. Origin is parameterised via xacro args so
-       real_bringup can plug in calibrated values from camera_pose.yaml
-       at launch time. -->
-  <xacro:macro name="volcaniarm_camera_joint">
+  <!-- camera_joint mounts the on-robot camera on camera_mount_rev_link
+       in normal mode (sim and real). In calibration mode the camera is
+       physically off the robot, so calibration_camera_joint in
+       volcaniarm_realsense.xacro parents camera_link directly to
+       base_link and this joint is skipped. The camera_x/y/z/roll/pitch/yaw
+       args parameterise the on-robot offset for a future eye-in-hand
+       calibration; defaults reflect the as-built mount. -->
+  <xacro:unless value="$(arg calibration)">
     <joint name="camera_joint" type="fixed">
       <origin xyz="$(arg camera_x) $(arg camera_y) $(arg camera_z)"
@@ -675,13 +679,5 @@
       <child link="camera_link" />
     </joint>
-  </xacro:macro>
-  <xacro:unless value="$(arg use_sim)">
-    <xacro:volcaniarm_camera_joint />
   </xacro:unless>
-  <xacro:if value="$(arg use_sim)">
-    <xacro:unless value="$(arg calibration)">
-      <xacro:volcaniarm_camera_joint />
-    </xacro:unless>
-  </xacro:if>
   <!-- Camera optical frame -->
   <link name="camera_link_optical" />

File: src/volcaniarm_description/urdf/volcaniarm_realsense.xacro (robot description, xacro)
@@ -1,32 +1,28 @@
 <?xml version="1.0"?>
 <robot xmlns:xacro="http://www.ros.org/wiki/xacro" name="volcaniarm_realsense">
-  <!-- Calibration mode: horizontal camera in front of the robot (sim only).
-       base_link is at world (0,0,0.98) with yaw=pi, so base_link +X is
-       world -X. xyz=(2.5, 0, -0.07) -> world (-2.5, 0, 0.91); yaw=pi
-       points +X back toward world +X.
-       Camera Z (0.91 m) is the midpoint of the workspace vertical
-       range (home tip near world Z=0.23, high targets near Z=1.58),
-       and the X distance (2.5 m) is set so the sim camera vertical
-       FOV of ~45 deg covers the full 1.55 m workspace span (with
-       0.2 m tag size accounted for) and keeps the entire EE tag
-       inside the image at every test pose. At 2 m distance the FOV
-       was ~0.24 m short and high-target captures lost the EE tag
-       to the top of the frame; pulling the camera back trades a
-       smaller tag in the image (~48 px wide vs ~62) for full
-       coverage of the operating envelope. -->
-  <!-- Sim-only override for calibration mode: parks the camera 1.5 m
-       in front of the robot facing back so the Gazebo workspace test
-       has a fixed view. On real hardware the camera is mounted on
-       the cart and the URDF's camera_joint (volcaniarm.urdf.xacro)
-       handles the placement, with calibrated values passed via xacro
-       args. -->
-  <xacro:if value="$(arg use_sim)">
-    <xacro:if value="$(arg calibration)">
-      <joint name="calibration_camera_joint" type="fixed">
-        <origin xyz="1.5 0 -0.5" rpy="0 0 ${pi}" />
-        <parent link="base_link" />
-        <child link="camera_link" />
-      </joint>
-    </xacro:if>
+  <!-- Calibration mode places the camera on an external stand, off the
+       robot, so it can see the full workspace plus the base tag in one
+       view. calibration_camera_joint parents camera_link directly to
+       world (skipping the on-robot mount) at a parameterised pose;
+       real_bringup forwards the calibrated values from camera_pose.yaml
+       so the URDF directly reflects the measured stand pose. Defaults
+       place the stand 1.5 m in front of the arm and 0.6 m above the
+       floor. Note: world_to_base has yaw=pi, so the arm reaches into
+       world -X. "In front of the arm" is world x=-1.5, with the
+       camera looking back toward world +X (rpy=0 since camera_link
+       inherits world's identity orientation). -->
+  <xacro:arg name="calibration_camera_x"     default="-1.5" />
+  <xacro:arg name="calibration_camera_y"     default="0.0" />
+  <xacro:arg name="calibration_camera_z"     default="0.6" />
+  <xacro:arg name="calibration_camera_roll"  default="0.0" />
+  <xacro:arg name="calibration_camera_pitch" default="0.0" />
+  <xacro:arg name="calibration_camera_yaw"   default="0.0" />
+  <xacro:if value="$(arg calibration)">
+    <joint name="calibration_camera_joint" type="fixed">
+      <origin xyz="$(arg calibration_camera_x) $(arg calibration_camera_y) $(arg calibration_camera_z)"
+              rpy="$(arg calibration_camera_roll) $(arg calibration_camera_pitch) $(arg calibration_camera_yaw)" />
+      <parent link="world" />
+      <child link="camera_link" />
+    </joint>
   </xacro:if>
   <!-- RealSense D435i frame chain. Published by robot_state_publisher in all
