Commit message: Replace camera calibration runners with mode-aware EE-sweep
Adds `mode:=work|tests` launch arg, orthogonal to `calibration`. The
four (mode, calibration) configurations now address: standard work,
on-robot camera pose calibration, full test workflow, and stand-camera
pose calibration. URDF gates camera parent and marker mounting on these
two args independently.

Replaces the single-shot localizer (camera_calibration.py) and the
full-6-DoF stand hand-eye runner (hand_eye_calibration.py) with one
EE-sweep runner that auto-detects mode from the URDF parent of
camera_link: `world` -> position-only solve (stand), `camera_mount_rev_link`
-> full 6-DoF cv2.calibrateHandEye eye-to-hand solve (on-robot). Both
modes share the 11 poses in calibration_poses.yaml, the sweep loop, and
write to a mode-keyed config/camera_pose.yaml that real_bringup applies
on launch.

Dashboard widget reads a `camera_calibration_only` parameter (set by the
launch when calibration:=true) to hide the test-runner panels and show
only the Camera localization group, plus a live Mode label tied to TF.
Pointcloud default flipped to true for parity with sim and to match
typical work-mode usage.

File: src/volcaniarm_description/urdf/volcaniarm.urdf.xacro (robot description, xacro)
@@ -2,4 +2,14 @@
 <robot xmlns:xacro="http://www.ros.org/wiki/xacro" name="volcaniarm">
   <xacro:arg name="use_sim" default="true" />
+  <!-- Physical configuration of the camera. Decoupled from `calibration`
+       so the four (mode, calibration) configurations are addressable:
+         mode=work,  calibration=false  -> normal working real hardware, no markers
+         mode=work,  calibration=true   -> on-robot camera + EE marker (calibrate camera_joint)
+         mode=tests, calibration=false  -> stand camera + both markers (accuracy / repeatability tests)
+         mode=tests, calibration=true   -> stand camera + EE marker (calibrate calibration_camera_joint) -->
+  <xacro:arg name="mode" default="work" />
+  <!-- Calibration overlay: when true, the calibration dashboard is up and
+       the EE marker is mounted. When false the markers + dashboard are
+       skipped (except in tests-mode where the test workflow needs both). -->
   <xacro:arg name="calibration" default="false" />
   <xacro:arg name="camera_mount_x" default="0.25" />
@@ -39,6 +49,22 @@
   <!-- Include RealSense camera frames for real hardware -->
   <xacro:include filename="$(find volcaniarm_description)/urdf/volcaniarm_realsense.xacro" />
-  <!-- Include AprilTag on EE for calibration in simulation -->
-  <xacro:if value="$(arg calibration)">
+  <!-- Marker configuration:
+         Base marker mounted whenever mode=tests (stand camera frames the
+           full workspace, so the base tag is in view and useful as a
+           fixed-frame reference for both the test workflow and the
+           camera-pose calibration sanity check).
+         EE marker mounted whenever mode=tests OR calibration=true
+           (so it's there for the on-robot calibration too, which has
+           no base marker).
+       The combined predicate `any_marker` decides whether the
+       apriltag.xacro file is even included; the per-marker xacro args
+       gate which links inside the file get instantiated. -->
+  <xacro:property name="mount_ee_marker"
+    value="${'$(arg calibration)' == 'true' or '$(arg mode)' == 'tests'}" />
+  <xacro:property name="mount_base_marker"
+    value="${'$(arg mode)' == 'tests'}" />
+  <xacro:property name="any_marker"
+    value="${mount_ee_marker or mount_base_marker}" />
+  <xacro:if value="${any_marker}">
     <xacro:include filename="$(find volcaniarm_description)/urdf/volcaniarm_apriltag.xacro" />
   </xacro:if>
@@ -579,9 +605,11 @@
   </joint>
   <!-- ======================== CAMERA MOUNT ======================== -->
-  <!-- Skipped in calibration mode: the camera is physically removed from
-       the robot and placed on an external stand, so calibration_camera_joint
-       in volcaniarm_realsense.xacro parents camera_link directly to
-       base_link instead. -->
-  <xacro:unless value="$(arg calibration)">
+  <!-- Active in work mode (camera physically on the robot). Skipped in
+       tests mode: the camera is on an external stand and
+       calibration_camera_joint in volcaniarm_realsense.xacro parents
+       camera_link directly to world instead. -->
+  <xacro:property name="camera_on_robot"
+    value="${'$(arg mode)' == 'work'}" />
+  <xacro:if value="${camera_on_robot}">
   <link name="camera_mount_linear_link">
     <inertial>
@@ -640,5 +668,5 @@
     <child link="camera_mount_rev_link" />
   </joint>
-  </xacro:unless>
+  </xacro:if>
   <!-- ======================== CAMERA ======================== -->
   <link name="camera_link">
@@ -666,11 +694,11 @@
   </link>
   <!-- camera_joint mounts the on-robot camera on camera_mount_rev_link
-       in normal mode (sim and real). In calibration mode the camera is
+       in work mode (sim and real). In tests mode the camera is
        physically off the robot, so calibration_camera_joint in
        volcaniarm_realsense.xacro parents camera_link directly to
-       base_link and this joint is skipped. The camera_x/y/z/roll/pitch/yaw
-       args parameterise the on-robot offset for a future eye-in-hand
-       calibration; defaults reflect the as-built mount. -->
-  <xacro:unless value="$(arg calibration)">
+       world and this joint is skipped. The camera_x/y/z/roll/pitch/yaw
+       args parameterise the on-robot offset and are written by the
+       camera-pose calibration's mode B (on_robot_mount). -->
+  <xacro:if value="${camera_on_robot}">
     <joint name="camera_joint" type="fixed">
       <origin xyz="$(arg camera_x) $(arg camera_y) $(arg camera_z)"
@@ -679,5 +707,5 @@
       <child link="camera_link" />
     </joint>
-  </xacro:unless>
+  </xacro:if>
   <!-- Camera optical frame -->
   <link name="camera_link_optical" />

File: src/volcaniarm_description/urdf/volcaniarm_apriltag.xacro (robot description, xacro)
@@ -1,11 +1,15 @@
 <?xml version="1.0"?>
 <robot xmlns:xacro="http://www.ros.org/wiki/xacro" name="volcaniarm_apriltag">
-  <!-- AprilTag 36h11 markers used for hand-eye calibration and accuracy
-       tests. Both tags use a DAE mesh with baked texture so they render
-       in Gazebo and RViz. The DAE geometry is 64 mm; the actual rendered
-       size follows the `tag_size` xacro arg (default 0.064 m, i.e. no
-       scaling), with the mesh scaled proportionally. Pass
-       tag_size:=0.200 in the launch file when using the larger printed
-       tags. -->
+  <!-- AprilTag 36h11 markers used for camera-pose calibration and the
+       test workflow (accuracy / repeatability). Both tags use a DAE
+       mesh with baked texture so they render in Gazebo and RViz. The
+       DAE geometry is 64 mm; the actual rendered size follows the
+       `tag_size` xacro arg (default 0.064 m, i.e. no scaling), with the
+       mesh scaled proportionally. Pass tag_size:=0.200 in the launch
+       file when using the larger printed tags.
+       Each marker is gated independently:
+         mount_ee_marker   - EE marker (ID 20) on right_arm_tip_link
+         mount_base_marker - base marker (ID 5) on volcaniarm_base_link
+       The parent xacro derives both flags from (mode, calibration). -->
   <xacro:property name="tag_size" value="$(arg tag_size)" />
   <xacro:property name="tag_scale" value="${tag_size / 0.064}" />
@@ -13,4 +17,5 @@
   <!-- ID 20: end-effector marker (right_arm_tip_link)                -->
   <!-- ============================================================= -->
+  <xacro:if value="${mount_ee_marker}">
   <xacro:property name="ee_tag_mesh"
     value="package://volcaniarm_description/models/Apriltag36_11_00020/apriltag_36h11_id20.dae" />
@@ -62,7 +67,9 @@
     <preserveFixedJoint>true</preserveFixedJoint>
   </gazebo>
+  </xacro:if>  <!-- mount_ee_marker -->
   <!-- ============================================================= -->
   <!-- ID 5: base-link reference marker (volcaniarm_base_link)        -->
   <!-- ============================================================= -->
+  <xacro:if value="${mount_base_marker}">
   <xacro:property name="base_tag_mesh"
     value="package://volcaniarm_description/models/Apriltag36_11_00005/apriltag_36h11_id05.dae" />
@@ -108,3 +115,4 @@
     <preserveFixedJoint>true</preserveFixedJoint>
   </gazebo>
+  </xacro:if>  <!-- mount_base_marker -->
 </robot>

File: src/volcaniarm_description/urdf/volcaniarm_realsense.xacro (robot description, xacro)
@@ -1,8 +1,8 @@
 <?xml version="1.0"?>
 <robot xmlns:xacro="http://www.ros.org/wiki/xacro" name="volcaniarm_realsense">
-  <!-- Calibration mode places the camera on an external stand, off the
-       robot, so it can see the full workspace plus the base tag in one
-       view. calibration_camera_joint parents camera_link directly to
-       world (skipping the on-robot mount) at a parameterised pose;
+  <!-- Tests mode places the camera on an external stand, off the robot,
+       so it can see the full workspace plus the base tag in one view.
+       calibration_camera_joint parents camera_link directly to world
+       (skipping the on-robot mount) at a parameterised pose;
        real_bringup forwards the calibrated values from camera_pose.yaml
        so the URDF directly reflects the measured stand pose. Defaults
@@ -18,5 +18,5 @@
   <xacro:arg name="calibration_camera_pitch" default="0.0" />
   <xacro:arg name="calibration_camera_yaw"   default="0.0" />
-  <xacro:if value="$(arg calibration)">
+  <xacro:if value="${'$(arg mode)' == 'tests'}">
     <joint name="calibration_camera_joint" type="fixed">
       <origin xyz="$(arg calibration_camera_x) $(arg calibration_camera_y) $(arg calibration_camera_z)"

Commit message: phase3: rebuild MoveIt on the phantom-chain approach (working reference)
Replace the custom-IK-on-the-closed-loop design with the phantom-chain approach
proven in the reference repo, but reuse our analytic volcaniarm_kinematics
(no urdfdom fork / Pinocchio):

- volcaniarm_description: new volcaniarm_moveit.xacro adds an OPEN phantom chain
  (prismatic tool_joint_y/z -> tool0) placing tool0 at the home EE
  (0.291, 0, 0.7489); gated by a new planning:=true xacro arg, off for the
  real/sim model.
- volcaniarm_moveit_config: SRDF group 'ee' = chain(base -> tool0) with the five
  real joints passive; kinematics.yaml -> stock KDL (no custom plugin);
  moveit_controllers -> the joint_state_transformer FJT controller; OMPL
  pipeline (defaults to RRTConnect, so no empty-planner_id failure); joint_limits
  for the phantom joints.
- New joint_state_transformer node: MoveIt executes the planned phantom (EE Y-Z)
  trajectory to it; it solves inverse_ee per waypoint and forwards to the JTC,
  and publishes the phantom joints (from the real elbows via forward_ee) so
  MoveIt tracks the actual EE.
- Retire the custom volcaniarm_ik_plugin and the Pilz configs.

Result: the RViz goal marker is inherently Y-Z only (the plan chain has only Y/Z
prismatic DOF), home is clean, and planning/execute work with stock KDL+OMPL.
Phases 1-2 (kinematics lib, broadcaster, oracle, pybind) are reused untouched.

File: src/volcaniarm_description/urdf/volcaniarm.urdf.xacro (robot description, xacro)
@@ -38,4 +38,8 @@
        parameter when forwarded by the bringup launches. -->
   <xacro:arg name="tag_size" default="0.064" />
+  <!-- MoveIt planning render: add the open phantom Y-Z chain to tool0 so MoveIt
+       can plan the (otherwise unplannable) closed loop. Only enabled for the
+       move_group robot_description; the real/sim model leaves it off. -->
+  <xacro:arg name="planning" default="false" />
   <!-- Camera mount position tuning
        camera_mount_x range: 0.155 to 0.655
@@ -69,4 +73,8 @@
     <xacro:include filename="$(find volcaniarm_description)/urdf/volcaniarm_apriltag.xacro" />
   </xacro:if>
+  <!-- MoveIt phantom planning chain (volcaniarm_base_link -> tool0); off by default. -->
+  <xacro:if value="$(arg planning)">
+    <xacro:include filename="$(find volcaniarm_description)/urdf/volcaniarm_moveit.xacro" />
+  </xacro:if>
   <!-- World fixed link -->
   <link name="world" />

File: src/volcaniarm_moveit_config/srdf/volcaniarm.srdf.xacro (robot description, xacro)
@@ -1,25 +1,29 @@
 <?xml version="1.0"?>
+<!-- Semantic description for MoveIt planning of the Volcaniarm five-bar.
+     MoveIt plans the OPEN phantom chain (volcaniarm_base_link -> tool0 via the
+     prismatic tool_joint_y/z); the joint_state_transformer node converts the
+     planned tool pose into the real elbow angles (inverse_ee) for execution.
+     The five real loop joints are passive (MoveIt never commands them). -->
 <robot xmlns:xacro="http://www.ros.org/wiki/xacro" name="volcaniarm">
-  <!--
-    Planning group for the planar five-bar. It is a two-branch closed loop, so
-    the group combines the right-branch chain (base -> right_arm_tip_link, the IK
-    tip) with the left-branch joints + closure, giving all five loop joints. The
-    three passive joints are marked <passive_joint>; only the two elbows are
-    actuated and executed by the JTC.
-  -->
-  <group name="volcaniarm">
-    <chain base_link="volcaniarm_base_link" tip_link="right_arm_tip_link"/>
-    <joint name="volcaniarm_left_elbow_joint"/>
-    <joint name="volcaniarm_left_arm_joint"/>
-    <joint name="closure_joint"/>
+  <!-- Planning group: the 2-DOF phantom chain positioning the EE point tool0. -->
+  <group name="ee">
+    <chain base_link="volcaniarm_base_link" tip_link="tool0"/>
   </group>
+  <!-- Home = q=0 assembly. The phantom origins put tool0 on the home EE when both
+       phantom joints are 0, so the default state is home and the goal marker
+       starts exactly on the EE. -->
+  <group_state name="home" group="ee">
+    <joint name="tool_joint_y" value="0.0"/>
+    <joint name="tool_joint_z" value="0.0"/>
+  </group_state>
+  <!-- The real linkage joints are driven by the loop closure / the transformer,
+       never commanded directly by MoveIt. -->
+  <passive_joint name="volcaniarm_left_elbow_joint"/>
+  <passive_joint name="volcaniarm_right_elbow_joint"/>
   <passive_joint name="volcaniarm_left_arm_joint"/>
   <passive_joint name="volcaniarm_right_arm_joint"/>
   <passive_joint name="closure_joint"/>
-  <group_state name="home" group="volcaniarm">
-    <joint name="volcaniarm_left_elbow_joint" value="0"/>
-    <joint name="volcaniarm_right_elbow_joint" value="0"/>
-  </group_state>
-  <!-- Adjacent links (connected by a joint) never meaningfully self-collide. -->
+  <!-- Disable the permanently-closed loop link pairs so the mechanism is not
+       flagged as self-colliding during phantom planning. -->
   <disable_collisions link1="volcaniarm_base_link" link2="volcaniarm_left_elbow_link" reason="Adjacent"/>
   <disable_collisions link1="volcaniarm_base_link" link2="volcaniarm_right_elbow_link" reason="Adjacent"/>
@@ -28,11 +32,8 @@
   <disable_collisions link1="volcaniarm_left_arm_link" link2="closure_dummy_link" reason="Adjacent"/>
   <disable_collisions link1="volcaniarm_right_arm_link" link2="right_arm_tip_link" reason="Adjacent"/>
-  <!-- The closure pin: these two leaves coincide by construction. -->
   <disable_collisions link1="closure_dummy_link" link2="right_arm_tip_link" reason="Closure"/>
   <disable_collisions link1="closure_dummy_link" link2="volcaniarm_right_arm_link" reason="Closure"/>
   <disable_collisions link1="right_arm_tip_link" link2="volcaniarm_left_arm_link" reason="Closure"/>
-  <!-- The two arm links meet at the closure point. -->
   <disable_collisions link1="volcaniarm_left_arm_link" link2="volcaniarm_right_arm_link" reason="Closure"/>
-  <!-- Base sits between the two elbows. -->
   <disable_collisions link1="volcaniarm_left_elbow_link" link2="volcaniarm_right_elbow_link" reason="Never"/>
 </robot>
